File: pilot/pilot.kicad_sch (KiCad schematic)
At the start: 0 parts

Commit message: 25/12/04
Other:
- added sheet rp2350a (rp2350a.kicad_sch)
Changed lines of the file:
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@@
 	(generator_version "9.0")
 	(paper "A4")
+	(sheet
+		(at 128.27 90.17)
+		(size 26.67 22.86)
+		(exclude_from_sim no)
+		(in_bom yes)
+		(on_board yes)
+		(dnp no)
+		(fields_autoplaced yes)
+		(stroke
+			(width 0.1524)
+			(type solid)
+		)
+		(fill
+			(color 0 0 0 0.0000)
+		)
+		(property "Sheetname" "rp2350a"
+			(at 128.27 89.4584 0)
+			(effects
+				(font
+					(size 1.27 1.27)
+				)
+				(justify left bottom)
+			)
+		)
+		(property "Sheetfile" "rp2350a.kicad_sch"
+			(at 128.27 113.6146 0)
+			(effects
+				(font
+					(size 1.27 1.27)
+				)
+				(justify left top)
+			)
+		)
+		(instances
+			(project "pilot"
+				(path "/6e01a02a-937c-45ab-a43c-49a8d1056ac9"
+					(page "2")
+				)
+			)
+		)
+	)
 	(sheet_instances
 		(path "/"

Commit message: 25/12/05/1234
Other:
- added sheet CAN (CAN.kicad_sch)
Changed lines of the file:
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@@
 	(paper "A4")
+	(sheet
+		(at 180.34 90.17)
+		(size 29.21 22.86)
+		(exclude_from_sim no)
+		(in_bom yes)
+		(on_board yes)
+		(dnp no)
+		(fields_autoplaced yes)
+		(stroke
+			(width 0.1524)
+			(type solid)
+		)
+		(fill
+			(color 0 0 0 0.0000)
+		)
+		(property "Sheetname" "CAN"
+			(at 180.34 89.4584 0)
+			(effects
+				(font
+					(size 1.27 1.27)
+				)
+				(justify left bottom)
+			)
+		)
+		(property "Sheetfile" "CAN.kicad_sch"
+			(at 180.34 113.6146 0)
+			(effects
+				(font
+					(size 1.27 1.27)
+				)
+				(justify left top)
+			)
+		)
+		(instances
+			(project "pilot"
+				(path "/6e01a02a-937c-45ab-a43c-49a8d1056ac9"
+					(page "3")
+				)
+			)
+		)
+	)
 	(sheet
 		(at 128.27 90.17)

Commit message: 2025/12/05/1722
初めてのコミット
Other:
- removed sheet CAN
- added sheet can (can.kicad_sch)
Changed lines of the file:
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@@
 	(paper "A4")
 	(sheet
-		(at 180.34 90.17)
-		(size 29.21 22.86)
+		(at 171.45 78.74)
+		(size 52.07 34.29)
 		(exclude_from_sim no)
 		(in_bom yes)
@@
 			(color 0 0 0 0.0000)
 		)
-		(property "Sheetname" "CAN"
-			(at 180.34 89.4584 0)
+		(property "Sheetname" "can"
+			(at 171.45 78.0284 0)
 			(effects
 				(font
@@
 			)
 		)
-		(property "Sheetfile" "CAN.kicad_sch"
-			(at 180.34 113.6146 0)
+		(property "Sheetfile" "can.kicad_sch"
+			(at 171.45 113.6146 0)
 			(effects
 				(font

Commit message: 25/12/08/1749
Parts:
- added C18, C19: 10u, symbol Device:C
- added J2: RJ45_Shielded, symbol Connector:RJ45_Shielded
- added J3: 電源入力, symbol Connector_Generic:Conn_01x02
- added U3: NCP1117-5.0_SOT223, Package_TO_SOT_SMD:SOT-223-3_TabPin2, symbol Regulator_Linear:NCP1117-5.0_SOT223
Connections:
- new net: C19.1, J3.2 (Pin_2), U3.3 (VI)
- new net CAN_H: J2.2
- new net CAN_L: J2.1
- new net GND: C18.2, C19.2, J2.3, J2.5, J2.7, J2.SH, J3.1 (Pin_1), U3.1 (GND)
- new net LAN_5V: J2.4, J2.6, J2.8
- new net imput_5V: C18.1, U3.2 (VO)
Other:
- removed sheet can
- added sheet CAN (CAN.kicad_sch)
- sheet rp2350a ports: added Input_5V, LAN_5V; removed none

Commit message: 2025/12/08/1826
Other:
- sheet rp2350a ports: added ELE_ADC, LAD_ADC; removed none
Changed lines of the file:
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@@
+			)
+		)
+		(pin "ELE_ADC" input
+			(at 154.94 81.28 0)
+			(effects
+				(font
+					(size 1.27 1.27)
+				)
+				(justify right)
+			)
+		)
+		(pin "LAD_ADC" input
+			(at 154.94 86.36 0)
+			(effects
+				(font
+					(size 1.27 1.27)
+				)
+				(justify right)
 			)
 		)
