File: pilot/pilot.kicad_sch (KiCad schematic)
At the start: 5 parts, among them J2 RJ45_Shielded, J3 電源入力, U3 NCP1117-5.0_SOT223

Commit message: 12/12
Other:
- sheet CAN ports: added CS, INT, SCK, SI, SO, VCC_CAN_CON; removed none
Changed lines of the file:
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@@
+			)
+		)
+		(pin "CS" input
+			(at 180.34 92.71 180)
+			(effects
+				(font
+					(size 1.27 1.27)
+				)
+				(justify left)
+			)
+		)
+		(pin "INT" input
+			(at 180.34 96.52 180)
+			(effects
+				(font
+					(size 1.27 1.27)
+				)
+				(justify left)
+			)
+		)
+		(pin "SCK" input
+			(at 180.34 100.33 180)
+			(effects
+				(font
+					(size 1.27 1.27)
+				)
+				(justify left)
+			)
+		)
+		(pin "SI" input
+			(at 180.34 104.14 180)
+			(effects
+				(font
+					(size 1.27 1.27)
+				)
+				(justify left)
+			)
+		)
+		(pin "SO" input
+			(at 180.34 107.95 180)
+			(effects
+				(font
+					(size 1.27 1.27)
+				)
+				(justify left)
+			)
+		)
+		(pin "VCC_CAN_CON" input
+			(at 180.34 111.76 180)
+			(effects
+				(font
+					(size 1.27 1.27)
+				)
+				(justify left)
 			)
 		)
@@
 	(sheet
 		(at 90.17 72.39)
-		(size 48.26 41.91)
+		(size 64.77 63.5)
 		(exclude_from_sim no)
 		(in_bom yes)
@@
 		)
 		(property "Sheetfile" "rp2350a.kicad_sch"
-			(at 90.17 114.8846 0)
+			(at 90.17 136.4746 0)
 			(effects
 				(font
@@
 		)
 		(pin "ELE_ADC" input
-			(at 138.43 81.28 0)
+			(at 154.94 81.28 0)
 			(effects
 				(font
@@
 		)
 		(pin "LAD_ADC" input
-			(at 138.43 86.36 0)
+			(at 154.94 86.36 0)
 			(effects
 				(font

Commit message: 2026/02/11/2106
Parts:
- added D5: D, symbol Device:D
- added J5, J6, J7: Conn_01x03, symbol Connector_Generic:Conn_01x03
- added J8: Conn_01x05, symbol Connector_Generic:Conn_01x05
- added J9: Conn_01x04, symbol Connector_Generic:Conn_01x04
- renumbered C19 to C1, C18 to C2, J2 to J1, J3 to J2, U3 to U1
Connections:
- net GND: now also J5.3 (Pin_3), J6.3 (Pin_3), J7.3 (Pin_3), J8.5 (Pin_5), J9.4 (Pin_4)
- new net: D5.2 (A), J8.1 (Pin_1)
- new net +3V3: D5.1 (K), J5.2 (Pin_2), J6.2 (Pin_2), J7.2 (Pin_2), J9.3 (Pin_3)
- new net DISPLAY_SCL: J9.1 (Pin_1)
- new net DISPLAY_SDA: J9.2 (Pin_2)
- new net ELE_ADC: J5.1 (Pin_1)
- new net LAD_ADC: J6.1 (Pin_1)
- new net SIM_SCL: J8.4 (Pin_4)
- new net SIM_SDA: J8.3 (Pin_3)
- new net SPARE_ADC: J7.1 (Pin_1)
- no-connect marks 0 -> 1
Other:
- added sheet Buzzer (untitled.kicad_sch)
- sheet CAN ports: added CANH, CANL, CAN_VDD; removed VCC_CAN_CON
- sheet rp2350a ports: added Buzzer, CAN_CS, CAN_INT, CAN_MISO, CAN_MOSI, CAN_SCK, I2C0_SCL, I2C0_SDA, I2C1_SCL, I2C1_SDA, SPARE_ADC; removed none

Commit message: 2026/02/12/1628
Parts:
- C1, C2: footprint (none) -> Capacitor_SMD:C_0805_2012Metric
- D1: renamed from D5; footprint (none) -> Diode_SMD:D_SMA
- J1: footprint (none) -> Connector_RJ:RJ45_Amphenol_RJHSE538X
- J2: renamed from J5; footprint (none) -> Connector_JST:JST_XH_B3B-XH-AM_1x03_P2.50mm_Vertical
- J3: renamed from J6; footprint (none) -> Connector_JST:JST_XH_B3B-XH-AM_1x03_P2.50mm_Vertical
- J4: renamed from J7; footprint (none) -> Connector_JST:JST_XH_B3B-XH-AM_1x03_P2.50mm_Vertical
- J5: renamed from J8; footprint (none) -> Connector_JST:JST_XH_B5B-XH-AM_1x05_P2.50mm_Vertical
- J6: renamed from J9; footprint (none) -> Connector_JST:JST_XH_B4B-XH-AM_1x04_P2.50mm_Vertical
- J7: renamed from J2; footprint (none) -> Connector_JST:JST_VH_B2P-VH-FB-B_1x02_P3.96mm_Vertical
Changed lines of the file:
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@@
 		(dnp no)
 		(fields_autoplaced yes)
-		(property "Reference" "#PWR04"
+		(property "Reference" "#PWR013"
 			(at 48.26 40.64 0)
 			(effects
@@
 			(project ""
 				(path "/6e01a02a-937c-45ab-a43c-49a8d1056ac9"
-					(reference "#PWR04")
+					(reference "#PWR013")
 					(unit 1)
 				)
@@
 		(dnp no)
 		(fields_autoplaced yes)
-		(property "Reference" "#PWR053"
+		(property "Reference" "#PWR06"
 			(at 35.56 114.3 0)
 			(effects
@@
 			(project "pilot"
 				(path "/6e01a02a-937c-45ab-a43c-49a8d1056ac9"
-					(reference "#PWR053")
+					(reference "#PWR06")
 					(unit 1)
 				)
@@
 		(dnp no)
 		(fields_autoplaced yes)
-		(property "Reference" "#PWR051"
+		(property "Reference" "#PWR03"
 			(at 45.72 88.9 0)
 			(effects
@@
 			(project ""
 				(path "/6e01a02a-937c-45ab-a43c-49a8d1056ac9"
-					(reference "#PWR051")
+					(reference "#PWR03")
 					(unit 1)
 				)
@@
 		(dnp no)
 		(fields_autoplaced yes)
-		(property "Reference" "#PWR049"
+		(property "Reference" "#PWR02"
 			(at 35.56 86.36 0)
 			(effects
@@
 			(project ""
 				(path "/6e01a02a-937c-45ab-a43c-49a8d1056ac9"
-					(reference "#PWR049")
+					(reference "#PWR02")
 					(unit 1)
 				)
@@
 		(dnp no)
 		(fields_autoplaced yes)
-		(property "Reference" "#PWR054"
+		(property "Reference" "#PWR07"
 			(at 45.72 116.84 0)
 			(effects
@@
 			(project "pilot"
 				(path "/6e01a02a-937c-45ab-a43c-49a8d1056ac9"
-					(reference "#PWR054")
+					(reference "#PWR07")
 					(unit 1)
 				)
@@
 		(dnp no)
 		(fields_autoplaced yes)
-		(property "Reference" "#PWR056"
+		(property "Reference" "#PWR08"
 			(at 45.72 135.89 0)
 			(effects
@@
 			(project ""
 				(path "/6e01a02a-937c-45ab-a43c-49a8d1056ac9"
-					(reference "#PWR056")
+					(reference "#PWR08")
 					(unit 1)
 				)
@@
 		(dnp no)
 		(fields_autoplaced yes)
-		(property "Reference" "#PWR052"
+		(property "Reference" "#PWR05"
 			(at 45.72 102.87 0)
 			(effects
@@
 			(project "pilot"
 				(path "/6e01a02a-937c-45ab-a43c-49a8d1056ac9"
-					(reference "#PWR052")
+					(reference "#PWR05")
 					(unit 1)
 				)
@@
 			)
 		)
-		(property "Footprint" ""
+		(property "Footprint" "Capacitor_SMD:C_0805_2012Metric"
 			(at 120.3452 38.1 0)
 			(effects
@@
 			)
 		)
-		(property "Footprint" ""
+		(property "Footprint" "Capacitor_SMD:C_0805_2012Metric"
 			(at 93.6752 38.1 0)
 			(effects
@@
 		(dnp no)
 		(fields_autoplaced yes)
-		(property "Reference" "#PWR050"
+		(property "Reference" "#PWR04"
 			(at 35.56 100.33 0)
 			(effects
@@
 			(project "pilot"
 				(path "/6e01a02a-937c-45ab-a43c-49a8d1056ac9"
-					(reference "#PWR050")
+					(reference "#PWR04")
 					(unit 1)
 				)
@@
 		(on_board yes)
 		(dnp no)
-		(property "Reference" "J5"
+		(property "Reference" "J2"
 			(at 31.75 85.0899 0)
 			(effects
@@
 			)
 		)
-		(property "Footprint" ""
+		(property "Footprint" "Connector_JST:JST_XH_B3B-XH-AM_1x03_P2.50mm_Vertical"
 			(at 34.29 86.36 0)
 			(effects
@@
 			(project ""
 				(path "/6e01a02a-937c-45ab-a43c-49a8d1056ac9"
-					(reference "J5")
+					(reference "J2")
 					(unit 1)
 				)
@@
 		(dnp no)
 		(fields_autoplaced yes)
-		(property "Reference" "#PWR05"
+		(property "Reference" "#PWR015"
 			(at 77.47 39.37 0)
 			(effects
@@
 			(project ""
 				(path "/6e01a02a-937c-45ab-a43c-49a8d1056ac9"
-					(reference "#PWR05")
+					(reference "#PWR015")
 					(unit 1)
 				)
@@
 		(dnp no)
 		(fields_autoplaced yes)
-		(property "Reference" "#PWR06"
+		(property "Reference" "#PWR016"
 			(at 92.71 44.45 0)
 			(effects
@@
 			(project ""
 				(path "/6e01a02a-937c-45ab-a43c-49a8d1056ac9"
-					(reference "#PWR06")
+					(reference "#PWR016")
 					(unit 1)
 				)
@@
 		(dnp no)
 		(fields_autoplaced yes)
-		(property "Reference" "#PWR02"
+		(property "Reference" "#PWR011"
 			(at 48.26 30.48 0)
 			(effects
@@
 			(project "pilot"
 				(path "/6e01a02a-937c-45ab-a43c-49a8d1056ac9"
-					(reference "#PWR02")
+					(reference "#PWR011")
 					(unit 1)
 				)
@@
 		(dnp no)
 		(fields_autoplaced yes)
-		(property "Reference" "#PWR07"
+		(property "Reference" "#PWR017"
 			(at 107.95 44.45 0)
 			(effects
@@
 			(project ""
 				(path "/6e01a02a-937c-45ab-a43c-49a8d1056ac9"
-					(reference "#PWR07")
+					(reference "#PWR017")
 					(unit 1)
 				)
@@
 		(dnp no)
 		(fields_autoplaced yes)
-		(property "Reference" "#PWR08"
+		(property "Reference" "#PWR018"
 			(at 119.38 44.45 0)
 			(effects
@@
 			(project ""
 				(path "/6e01a02a-937c-45ab-a43c-49a8d1056ac9"
-					(reference "#PWR08")
+					(reference "#PWR018")
 					(unit 1)
 				)
@@
 		(dnp no)
 		(fields_autoplaced yes)
-		(property "Reference" "#PWR055"
+		(property "Reference" "#PWR014"
 			(at 48.26 125.73 0)
 			(effects
@@
 			(project ""
 				(path "/6e01a02a-937c-45ab-a43c-49a8d1056ac9"
-					(reference "#PWR055")
+					(reference "#PWR014")
 					(unit 1)
 				)
@@
 		(on_board yes)
 		(dnp no)
-		(property "Reference" "J6"
+		(property "Reference" "J3"
 			(at 31.75 99.0599 0)
 			(effects
@@
 			)
 		)
-		(property "Footprint" ""
+		(property "Footprint" "Connector_JST:JST_XH_B3B-XH-AM_1x03_P2.50mm_Vertical"
 			(at 34.29 100.33 0)
 			(effects
@@
 			(project "pilot"
 				(path "/6e01a02a-937c-45ab-a43c-49a8d1056ac9"
-					(reference "J6")
+					(reference "J3")
 					(unit 1)
 				)
@@
 		(dnp no)
 		(fields_autoplaced yes)
-		(property "Reference" "J2"
+		(property "Reference" "J7"
 			(at 72.39 24.13 0)
 			(effects
@@
 			)
 		)
-		(property "Footprint" ""
+		(property "Footprint" "Connector_JST:JST_VH_B2P-VH-FB-B_1x02_P3.96mm_Vertical"
 			(at 72.39 33.02 0)
 			(effects
@@
 			(project ""
 				(path "/6e01a02a-937c-45ab-a43c-49a8d1056ac9"
-					(reference "J2")
+					(reference "J7")
 					(unit 1)
 				)
@@
 		(on_board yes)
 		(dnp no)
-		(property "Reference" "J9"
+		(property "Reference" "J6"
 			(at 31.75 146.0499 0)
 			(effects
@@
 			)
 		)
-		(property "Footprint" ""
+		(property "Footprint" "Connector_JST:JST_XH_B4B-XH-AM_1x04_P2.50mm_Vertical"
 			(at 34.29 146.05 0)
 			(effects
@@
 			(project ""
 				(path "/6e01a02a-937c-45ab-a43c-49a8d1056ac9"
-					(reference "J9")
+					(reference "J6")
 					(unit 1)
 				)
@@
 		(on_board yes)
 		(dnp no)
-		(property "Reference" "D5"
+		(property "Reference" "D1"
 			(at 44.45 119.38 0)
 			(effects
@@
 			)
 		)
-		(property "Footprint" ""
+		(property "Footprint" "Diode_SMD:D_SMA"
 			(at 44.45 125.73 0)
 			(effects
@@
 			(project ""
 				(path "/6e01a02a-937c-45ab-a43c-49a8d1056ac9"
-					(reference "D5")
+					(reference "D1")
 					(unit 1)
 				)
@@
 		(dnp no)
 		(fields_autoplaced yes)
-		(property "Reference" "#PWR058"
+		(property "Reference" "#PWR010"
 			(at 45.72 151.13 0)
 			(effects
@@
 			(project ""
 				(path "/6e01a02a-937c-45ab-a43c-49a8d1056ac9"
-					(reference "#PWR058")
+					(reference "#PWR010")
 					(unit 1)
 				)
@@
 		(dnp no)
 		(fields_autoplaced yes)
-		(property "Reference" "#PWR057"
+		(property "Reference" "#PWR09"
 			(at 35.56 148.59 0)
 			(effects
@@
 			(project ""
 				(path "/6e01a02a-937c-45ab-a43c-49a8d1056ac9"
-					(reference "#PWR057")
+					(reference "#PWR09")
 					(unit 1)
 				)
@@
 			)
 		)
-		(property "Footprint" ""
+		(property "Footprint" "Connector_RJ:RJ45_Amphenol_RJHSE538X"
 			(at 31.75 37.465 90)
 			(effects
@@
 		(dnp no)
 		(fields_autoplaced yes)
-		(property "Reference" "#PWR09"
+		(property "Reference" "#PWR019"
 			(at 208.28 128.27 0)
 			(effects
@@
 			(project ""
 				(path "/6e01a02a-937c-45ab-a43c-49a8d1056ac9"
-					(reference "#PWR09")
+					(reference "#PWR019")
 					(unit 1)
 				)
@@
 		(on_board yes)
 		(dnp no)
-		(property "Reference" "J7"
+		(property "Reference" "J4"
 			(at 31.75 113.0299 0)
 			(effects
@@
 			)
 		)
-		(property "Footprint" ""
+		(property "Footprint" "Connector_JST:JST_XH_B3B-XH-AM_1x03_P2.50mm_Vertical"
 			(at 34.29 114.3 0)
 			(effects
@@
 			(project "pilot"
 				(path "/6e01a02a-937c-45ab-a43c-49a8d1056ac9"
-					(reference "J7")
+					(reference "J4")
 					(unit 1)
 				)
@@
 		(on_board yes)
 		(dnp no)
-		(property "Reference" "J8"
+		(property "Reference" "J5"
 			(at 31.75 129.5399 0)
 			(effects
@@
 			)
 		)
-		(property "Footprint" ""
+		(property "Footprint" "Connector_JST:JST_XH_B5B-XH-AM_1x05_P2.50mm_Vertical"
 			(at 34.29 130.81 0)
 			(effects
@@
 			(project ""
 				(path "/6e01a02a-937c-45ab-a43c-49a8d1056ac9"
-					(reference "J8")
+					(reference "J5")
 					(unit 1)
 				)
@@
 		(dnp no)
 		(fields_autoplaced yes)
-		(property "Reference" "#PWR03"
+		(property "Reference" "#PWR012"
 			(at 48.26 35.56 0)
 			(effects
@@
 			(project "pilot"
 				(path "/6e01a02a-937c-45ab-a43c-49a8d1056ac9"
-					(reference "#PWR03")
-					(unit 1)
-				)
+					(reference "#PWR012")
+					(unit 1)
+				)

Commit message: 2026/02/15
Connections:
- net CAN_H: now also J1.1; no longer J1.2
- net CAN_L: now also J1.2; no longer J1.1
Changed lines of the file:
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@@
 	)
 	(label "CAN_H"
-		(at 41.91 43.18 0)
+		(at 41.91 45.72 0)
 		(effects
 			(font
@@
 	)
 	(label "CAN_L"
-		(at 41.91 45.72 0)
-		(effects
-			(font
+		(at 41.91 43.18 0)
+		(effects
+			(font
