File: pilot/CAN.kicad_sch (KiCad schematic)
At the start: 0 parts

Commit message: 12/12
Parts:
- added C23, C24: 22, symbol Device:C
- added U5: MCP2515-xSO, Package_SO:SOIC-18W_7.5x11.6mm_P1.27mm, symbol Interface_CAN_LIN:MCP2515-xSO
- added Y3: ABLS-8.000MHZ-12-B-4-Y-T, ABLS8000MHz12B4YT, symbol ABLS-8_000MHZ-12-B-4-Y-T:ABLS-8.000MHZ-12-B-4-Y-T

Commit message: 12/12
Parts:
- added C25, C27: 100n, symbol Device:C
- added C26: 10u, symbol Device:C
- added C28: 15u, symbol Device:C
- added U6: MCP2551-I-SN, Package_SO:SOIC-8_3.9x4.9mm_P1.27mm, symbol Interface_CAN_LIN:MCP2551-I-SN
- C23, C24: value 22 -> 22p
Connections:
- net GND: now also C23.2, C24.2, U5.9 (VSS), C26.2, C27.2, C28.2, U6.2 (VSS), U6.8 (Rs)
- net at C23.1: now also U5.8 (OSC1), Y3.2
- net at C24.1: now also U5.7 (OSC2), Y3.1
- net at U5.1 (TXCAN): now also U6.1 (TXD)
- net VCC_CAN_CON: now reaches U5.18 (VDD)
- net VCC_CAN_CON: now also C26.1, C27.1
- net RXCAN: now reaches U5.2 (RXCAN)
- net RXCAN: now also U6.4 (RXD)
- new net +5V: C25.1, C28.1, U6.3 (VDD)

Commit message: 12/22
12/22
Parts:
- added C29: 100n, symbol Device:C
- added D4: D, symbol Device:D
- added R10, R9: 10k, symbol Device:R
- added R11: 120, symbol Device:R
Connections:
- net CS: now also U5.16 (~{CS})
- net GND: now also C29.2
- net INT: now also U5.12 (~{INT})
- net SCK: now also U5.13 (SCK)
- net SI: now also U5.14 (SI)
- net SO: now also U5.15 (SO)
- net VCC_CAN_CON: now also D4.1 (K), R9.2
- net at U5.17 (~{RESET}): now also R10.1
- net 2: now reaches U6.6 (CANL)
- net 2: now also R11.2
- net 1: now reaches U6.7 (CANH)
- net 1: now also R11.1
- new net RESET: C29.1, D4.2 (A), R10.2, R9.1

Commit message: 2026/02/11/1853
Parts:
- removed C28: 15u, symbol Device:C
- removed C29: 100n, symbol Device:C
- removed U6: MCP2551-I-SN, Package_SO:SOIC-8_3.9x4.9mm_P1.27mm, symbol Interface_CAN_LIN:MCP2551-I-SN
- added IC1: TJA1050T, SOIC127P600X175-8N, symbol TJA1050T:TJA1050T
- added J4, J5: Conn_01x02, symbol Connector_Generic:Conn_01x02
- C26: value 10u -> 100n
- C27: value 100n -> 10μF
- R11: value 120 -> 1K
- R9: value 10k -> 120
Connections:
- net 1 is gone; now on net CAN_VDD: R11.1
- net GND: now also C25.2, C26.1, D4.1 (K), IC1.2 (GND), IC1.8 (S); no longer C26.2
- net RXCAN: now also IC1.4 (RXD)
- net TXCAN: now reaches U5.1 (TXCAN)
- net TXCAN: now also IC1.1 (TXD)
- net +5V renamed CAN_VDD
- net CAN_VDD: now also C26.2, C27.1, R10.2, U5.18 (VDD), IC1.3 (VCC)
- net 2: no longer names the net of R11.2
- net 2: now also D4.2 (A)
- removed net RESET: D4.2 (A), R10.2, R9.1
- removed net VCC_CAN_CON: C26.1, C27.1, D4.1 (K), R9.2, U5.18 (VDD)
- new net: IC1.6 (CANL), J4.1 (Pin_1), J5.1 (Pin_1), R9.2
- new net: IC1.7 (CANH), J4.2 (Pin_2), J5.2 (Pin_2), R9.1
- no-connect marks 0 -> 7
Other:
- note added: "水晶発振子を使うこと。"
- moved on the sheet: R10

Commit message: 2026/02/11/2106
Parts:
- removed J4: Conn_01x02, symbol Connector_Generic:Conn_01x02
- Y2: renamed from Y3; footprint ABLS8000MHz12B4YT -> crystal:ABLS8000MHz12B4YT
- renumbered C24 to C23, C27 to C24, C23 to C25, C25 to C26, C26 to C27, J5 to J4, R9 to R11, R11 to R9
Connections:
- net CANL: now reaches IC1.6 (CANL), J4.1 (Pin_1), R11.2
- net CANH: now reaches IC1.7 (CANH), J4.2 (Pin_2), R11.1
Changed lines of the file:
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@@
+		)
+	)
+	(hierarchical_label "CANL"
+		(shape input)
+		(at 245.11 71.12 0)
+		(effects
+			(font
+				(size 1.27 1.27)
+			)
+			(justify left)
 		)
 	)
@@
 		)
 	)
+	(hierarchical_label "CANH"
+		(shape input)
+		(at 245.11 73.66 0)
+		(effects
+			(font
+				(size 1.27 1.27)
+			)
+			(justify left)
+		)
+	)
 	(hierarchical_label "SCK"
 		(shape input)
@@
 		(dnp no)
 		(fields_autoplaced yes)
-		(property "Reference" "#PWR037"
+		(property "Reference" "#PWR041"
 			(at 157.48 118.11 0)
 			(effects
@@
 			(project ""
 				(path "/6e01a02a-937c-45ab-a43c-49a8d1056ac9/dfd1c32f-bd86-4594-b3e8-9cea7250640c"
-					(reference "#PWR037")
-					(unit 1)
-				)
-			)
-		)
-	)
-	(symbol
-		(lib_id "Connector_Generic:Conn_01x02")
-		(at 250.19 71.12 0)
-		(unit 1)
-		(exclude_from_sim no)
-		(in_bom yes)
-		(on_board yes)
-		(dnp no)
-		(fields_autoplaced yes)
-		(property "Reference" "J4"
-			(at 252.73 71.1199 0)
-			(effects
-				(font
-					(size 1.27 1.27)
-				)
-				(justify left)
-			)
-		)
-		(property "Value" "Conn_01x02"
-			(at 252.73 73.6599 0)
-			(effects
-				(font
-					(size 1.27 1.27)
-				)
-				(justify left)
-			)
-		)
-		(property "Footprint" ""
-			(at 250.19 71.12 0)
-			(effects
-				(font
-					(size 1.27 1.27)
-				)
-				(hide yes)
-			)
-		)
-		(property "Datasheet" "~"
-			(at 250.19 71.12 0)
-			(effects
-				(font
-					(size 1.27 1.27)
-				)
-				(hide yes)
-			)
-		)
-		(property "Description" "Generic connector, single row, 01x02, script generated (kicad-library-utils/schlib/autogen/connector/)"
-			(at 250.19 71.12 0)
-			(effects
-				(font
-					(size 1.27 1.27)
-				)
-				(hide yes)
-			)
-		)
-		(pin "1"
-		)
-		(pin "2"
-		)
-		(instances
-			(project ""
-				(path "/6e01a02a-937c-45ab-a43c-49a8d1056ac9/dfd1c32f-bd86-4594-b3e8-9cea7250640c"
-					(reference "J4")
+					(reference "#PWR041")
 					(unit 1)
 				)
@@
 		(dnp no)
 		(fields_autoplaced yes)
-		(property "Reference" "R9"
+		(property "Reference" "R11"
 			(at 241.3 57.1499 0)
 			(effects
@@
 			(project ""
 				(path "/6e01a02a-937c-45ab-a43c-49a8d1056ac9/dfd1c32f-bd86-4594-b3e8-9cea7250640c"
-					(reference "R9")
+					(reference "R11")
 					(unit 1)
 				)
@@
 		(dnp no)
 		(fields_autoplaced yes)
-		(property "Reference" "R11"
+		(property "Reference" "R9"
 			(at 114.3 31.7499 0)
 			(effects
@@
 			(project ""
 				(path "/6e01a02a-937c-45ab-a43c-49a8d1056ac9/dfd1c32f-bd86-4594-b3e8-9cea7250640c"
-					(reference "R11")
+					(reference "R9")
 					(unit 1)
 				)
@@
 		(dnp no)
 		(fields_autoplaced yes)
-		(property "Reference" "C23"
+		(property "Reference" "C25"
 			(at 105.41 105.4099 0)
 			(effects
@@
 			(project ""
 				(path "/6e01a02a-937c-45ab-a43c-49a8d1056ac9/dfd1c32f-bd86-4594-b3e8-9cea7250640c"
-					(reference "C23")
+					(reference "C25")
 					(unit 1)
 				)
@@
 		(dnp no)
 		(fields_autoplaced yes)
-		(property "Reference" "#PWR040"
+		(property "Reference" "#PWR043"
 			(at 176.53 78.74 0)
 			(effects
@@
 			(project ""
 				(path "/6e01a02a-937c-45ab-a43c-49a8d1056ac9/dfd1c32f-bd86-4594-b3e8-9cea7250640c"
-					(reference "#PWR040")
+					(reference "#PWR043")
 					(unit 1)
 				)
@@
 		(dnp no)
 		(fields_autoplaced yes)
-		(property "Reference" "C27"
+		(property "Reference" "C24"
 			(at 101.6 39.3699 0)
 			(effects
@@
 			(project ""
 				(path "/6e01a02a-937c-45ab-a43c-49a8d1056ac9/dfd1c32f-bd86-4594-b3e8-9cea7250640c"
-					(reference "C27")
+					(reference "C24")
 					(unit 1)
 				)
@@
 		(dnp no)
 		(fields_autoplaced yes)
-		(property "Reference" "C26"
+		(property "Reference" "C27"
 			(at 184.15 53.3399 0)
 			(effects
@@
 			(project ""
 				(path "/6e01a02a-937c-45ab-a43c-49a8d1056ac9/dfd1c32f-bd86-4594-b3e8-9cea7250640c"
-					(reference "C26")
+					(reference "C27")
 					(unit 1)
 				)
@@
 		(dnp no)
 		(fields_autoplaced yes)
-		(property "Reference" "#PWR038"
+		(property "Reference" "#PWR039"
 			(at 111.76 57.15 0)
 			(effects
@@
 			(project ""
 				(path "/6e01a02a-937c-45ab-a43c-49a8d1056ac9/dfd1c32f-bd86-4594-b3e8-9cea7250640c"
-					(reference "#PWR038")
+					(reference "#PWR039")
 					(unit 1)
 				)
@@
 		(dnp no)
 		(fields_autoplaced yes)
-		(property "Reference" "C24"
+		(property "Reference" "C23"
 			(at 92.71 105.4099 0)
 			(effects
@@
 			(project ""
 				(path "/6e01a02a-937c-45ab-a43c-49a8d1056ac9/dfd1c32f-bd86-4594-b3e8-9cea7250640c"
-					(reference "C24")
+					(reference "C23")
 					(unit 1)
 				)
@@
 		(dnp no)
 		(fields_autoplaced yes)
-		(property "Reference" "#PWR039"
+		(property "Reference" "#PWR037"
 			(at 97.79 57.15 0)
 			(effects
@@
 			(project "pilot"
 				(path "/6e01a02a-937c-45ab-a43c-49a8d1056ac9/dfd1c32f-bd86-4594-b3e8-9cea7250640c"
-					(reference "#PWR039")
+					(reference "#PWR037")
 					(unit 1)
 				)
@@
 		(dnp no)
 		(fields_autoplaced yes)
-		(property "Reference" "#PWR034"
+		(property "Reference" "#PWR038"
 			(at 101.6 120.65 0)
 			(effects
@@
 			(project ""
 				(path "/6e01a02a-937c-45ab-a43c-49a8d1056ac9/dfd1c32f-bd86-4594-b3e8-9cea7250640c"
-					(reference "#PWR034")
+					(reference "#PWR038")
 					(unit 1)
 				)
@@
 		(on_board yes)
 		(dnp no)
-		(property "Reference" "#PWR036"
+		(property "Reference" "#PWR042"
 			(at 180.34 44.45 0)
 			(effects
@@
 			(project ""
 				(path "/6e01a02a-937c-45ab-a43c-49a8d1056ac9/dfd1c32f-bd86-4594-b3e8-9cea7250640c"
-					(reference "#PWR036")
+					(reference "#PWR042")
 					(unit 1)
 				)
@@
 		(dnp no)
 		(fields_autoplaced yes)
-		(property "Reference" "J5"
+		(property "Reference" "J4"
 			(at 252.73 81.2799 0)
 			(effects
@@
 			(project "pilot"
 				(path "/6e01a02a-937c-45ab-a43c-49a8d1056ac9/dfd1c32f-bd86-4594-b3e8-9cea7250640c"
-					(reference "J5")
+					(reference "J4")
 					(unit 1)
 				)
@@
 		(dnp no)
 		(fields_autoplaced yes)
-		(property "Reference" "C25"
+		(property "Reference" "C26"
 			(at 161.29 106.6799 0)
 			(effects
@@
 			(project ""
 				(path "/6e01a02a-937c-45ab-a43c-49a8d1056ac9/dfd1c32f-bd86-4594-b3e8-9cea7250640c"
-					(reference "C25")
+					(reference "C26")
 					(unit 1)
 				)
@@
 		(dnp no)
 		(fields_autoplaced yes)
-		(property "Reference" "#PWR035"
+		(property "Reference" "#PWR036"
 			(at 88.9 120.65 0)
 			(effects
@@
 			(project ""
 				(path "/6e01a02a-937c-45ab-a43c-49a8d1056ac9/dfd1c32f-bd86-4594-b3e8-9cea7250640c"
-					(reference "#PWR035")
+					(reference "#PWR036")
 					(unit 1)
 				)
@@
 		(on_board yes)
 		(dnp no)
-		(property "Reference" "Y3"
+		(property "Reference" "Y2"
 			(at 82.296 94.996 0)
 			(effects
@@
 			)
 		)
-		(property "Footprint" "ABLS8000MHz12B4YT"
+		(property "Footprint" "crystal:ABLS8000MHz12B4YT"
 			(at 99.06 192.71 0)
 			(effects
@@
 			(project ""
 				(path "/6e01a02a-937c-45ab-a43c-49a8d1056ac9/dfd1c32f-bd86-4594-b3e8-9cea7250640c"
-					(reference "Y3")
+					(reference "Y2")
 					(unit 1)
 				)
@@
 		(dnp no)
 		(fields_autoplaced yes)
-		(property "Reference" "#PWR043"
+		(property "Reference" "#PWR040"
 			(at 132.08 119.38 0)
 			(effects
@@
 			(project ""
 				(path "/6e01a02a-937c-45ab-a43c-49a8d1056ac9/dfd1c32f-bd86-4594-b3e8-9cea7250640c"
-					(reference "#PWR043")
-					(unit 1)
-				)
+					(reference "#PWR040")
+					(unit 1)
+				)
