File: pilot/CAN.kicad_sch (KiCad schematic)
At the start: 13 parts, among them IC2 TJA1050T, J11 Conn_01x02, U4 MCP2515-xSO, Y2 ABLS-8.000MHZ-12-B-4-Y-T

Commit message: 20261001
Parts:
- D5: renamed from D6; footprint Diode_SMD:D_SMA -> LED_SMD:LED_0603_1608Metric
- renumbered R9 to R10, R10 to R11, R11 to R12
Changed lines of the file:
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@@
 		(dnp no)
 		(fields_autoplaced yes)
-		(property "Reference" "R11"
+		(property "Reference" "R12"
 			(at 241.3 57.1499 0)
 			(effects
@@
 			(project ""
 				(path "/6e01a02a-937c-45ab-a43c-49a8d1056ac9/dfd1c32f-bd86-4594-b3e8-9cea7250640c"
-					(reference "R11")
+					(reference "R12")
 					(unit 1)
 				)
@@
 		(dnp no)
 		(fields_autoplaced yes)
-		(property "Reference" "R9"
+		(property "Reference" "R10"
 			(at 114.3 31.7499 0)
 			(effects
@@
 			(project ""
 				(path "/6e01a02a-937c-45ab-a43c-49a8d1056ac9/dfd1c32f-bd86-4594-b3e8-9cea7250640c"
-					(reference "R9")
+					(reference "R10")
 					(unit 1)
 				)
@@
 		(dnp no)
 		(fields_autoplaced yes)
-		(property "Reference" "D6"
+		(property "Reference" "D5"
 			(at 114.3 43.1799 90)
 			(effects
@@
 			)
 		)
-		(property "Footprint" "Diode_SMD:D_SMA"
+		(property "Footprint" "LED_SMD:LED_0603_1608Metric"
 			(at 111.76 44.45 0)
 			(effects
@@
 			(project ""
 				(path "/6e01a02a-937c-45ab-a43c-49a8d1056ac9/dfd1c32f-bd86-4594-b3e8-9cea7250640c"
-					(reference "D6")
+					(reference "D5")
 					(unit 1)
 				)
@@
 		(dnp no)
 		(fields_autoplaced yes)
-		(property "Reference" "R10"
+		(property "Reference" "R11"
 			(at 151.13 95.25 90)
 			(effects
@@
 			(project ""
 				(path "/6e01a02a-937c-45ab-a43c-49a8d1056ac9/dfd1c32f-bd86-4594-b3e8-9cea7250640c"
-					(reference "R10")
-					(unit 1)
-				)
+					(reference "R11")
+					(unit 1)
+				)
