File: pilot/rp2350a.kicad_sch (KiCad schematic)
At the start: 4 parts, among them U1 RP2350_60QFN

Commit message: 25/12/05
Parts:
- added C3: 4,7u, symbol Device:C
- added L1: 3.3u, symbol Device:L
- C2: value C -> 4.7u
Connections:
- net GND: now also C2.2, U1.47 (VREG_PGND), C3.2
- net at U1.48 (VREG_LX): now also L1.2
- net -3V3: now reaches U1.49 (VREG_VIN)
- net -3V3: now also C2.1, R1.2
- net +1V1: now reaches U1.50 (VREG_FB)
- net +1V1: now also C3.1, L1.1

Commit message: 25/12/05/1234
Other:
- moved on the sheet: C1, C2, C3, L1, R1, U1

Commit message: 25/12/05/1637
Parts:
- added C4, C5: 10u, symbol Device:C
- added D1: D, symbol Device:D
- added J1: USB_B_Micro, symbol Connector:USB_B_Micro
- added U2: NCP1117-3.3_SOT223, Package_TO_SOT_SMD:SOT-223-3_TabPin2, symbol Regulator_Linear:NCP1117-3.3_SOT223
Connections:
- net GND: now also C4.2, C5.2, J1.5 (GND), J1.6 (Shield), U2.1 (GND)
- net -3V3 renamed +3.3V
- net +3.3V: now also C5.1, U2.2 (VO)
- new net: D1.2 (A), J1.1 (VBUS)
- new net USB_D+: J1.3 (D+)
- new net USB_D-: J1.2 (D-)
- new net VBUS: C4.1, D1.1 (K), U2.3 (VI)
- no-connect marks 0 -> 1
Other:
- note added: "power"

Commit message: 25/12/08/1749
Parts:
- added C10, C11, C12, C13, C14, C15, C16, C17, C6, C8, C9: 100n, symbol Device:C
- added C20: 100n, Capacitor_SMD:C_0402_1005Metric, symbol Device:C
- added C21, C22: 15p, Capacitor_SMD:C_0402_1005Metric, symbol Device:C
- added C7: 4,7u, symbol Device:C
- added D2, D3: D, symbol Device:D
- added R2, R3: 27, symbol Device:R
- added R4: 10k, Capacitor_SMD:C_0402_1005Metric, symbol Device:R
- added R5: 0, Capacitor_SMD:C_0402_1005Metric, symbol Device:R
- added R6, R7: 1k, Capacitor_SMD:C_0402_1005Metric, symbol Device:R
- added SW1: SW_Push, Button_Switch_SMD:SW_Push_1P1T_NO_Vertical_Wuerth_434133025816, symbol Switch:SW_Push
- added U4: W25Q128JVS, Package_SO:SOIC-8_5.23x5.23mm_P1.27mm, symbol Memory_Flash:W25Q128JVS
- added Y1: ABM8-272-T3, SamacSys_Parts:ABM8272T3, symbol SamacSys_Parts:ABM8-272-T3
Connections:
- net +3.3V is gone; now on net +3V3: C2.1, C5.1, R1.2, U1.49 (VREG_VIN), U2.2 (VO)
- net +1V1: now also U1.23 (DVDD), U1.39 (DVDD), U1.6 (DVDD), C6.1, C7.1, C8.1
- net GND: now also U1.61 (GND), C10.2, C11.2, C12.2, C13.2, C14.2, C15.2, C16.2, C17.2, C20.1, C21.2, C22.2, C6.2, C7.2, C8.2, C9.2, SW1.1, U4.4 (GND), Y1.2 (GND_1), Y1.4 (GND_2)
- net USB_D+: now also R2.1
- net USB_D-: now also R3.1
- net VBUS: now also D2.1 (K), D3.1 (K)
- net +3V3: now reaches U1.1 (IOVDD)
- net +3V3: now also U1.11 (IOVDD), U1.20 (IOVDD), U1.30 (IOVDD), U1.38 (IOVDD), U1.44 (ADC_AVDD), U1.45 (IOVDD), U1.53 (USB_OTP_VDD), U1.54 (QSPI_IOVDD), C10.1, C11.1, C12.1, C13.1, C14.1, C15.1, C16.1, C17.1, C20.2, C9.1, R4.2, U4.8 (VCC)
- net XIN: now reaches U1.21 (XIN)
- net XIN: now also C21.1, Y1.1 (CRYSTAL_1)
- net XOUT: now reaches U1.22 (XOUT)
- net XOUT: now also R7.1
- net at U1.51 (USB_DM): now also R3.2
- net at U1.52 (USB_DP): now also R2.2
- net QSPI_SD3: now reaches U1.55 (QSPI_SD3)
- net QSPI_SD3: now also U4.7 (IO3)
- net QSPI_SCLK: now reaches U1.56 (QSPI_SCLK)
- net QSPI_SCLK: now also U4.6 (CLK)
- net QSPI_SD0: now reaches U1.57 (QSPI_SD0)
- net QSPI_SD0: now also U4.5 (DI(IO0))
- net QSPI_SD2: now reaches U1.58 (QSPI_SD2)
- net QSPI_SD2: now also U4.3 (IO2)
- net QSPI_SD1: now reaches U1.59 (QSPI_SD1)
- net QSPI_SD1: now also U4.2 (DO(IO1))
- net QSPI_SS: now reaches U1.60 (QSPI_SS)
- net QSPI_SS: now also R5.2, R6.1
- new net: C22.1, R7.2, Y1.3 (CRYSTAL_2)
- new net GPIO0: R4.1, R5.1, U4.1 (~{CS})
- new net Input_5V: D3.2 (A)
- new net LAN_5V: D2.2 (A)
- new net ~{USB_BOOT}: R6.2, SW1.2
- no-connect marks 1 -> 3

Commit message: 2025/12/08/1826
Parts:
- added R8: 1k, symbol Device:R
- added SW2: SW_Push, symbol Switch:SW_Push
Connections:
- net GND: now also R8.2
- net at U1.26 (RUN): now also SW2.2
- net LAD_ADC: now reaches U1.40 (GPIO26_ADC0)
- net ELE_ADC: now reaches U1.41 (GPIO27_ADC1)
- net SPARE_ADC: now reaches U1.42 (GPIO28_ADC2)
- new net: R8.1, SW2.1

Commit message: 2026/02/11/2106
Parts:
- added J10: Conn_01x12, symbol Connector_Generic:Conn_01x12
- added J11: Conn_01x06, symbol Connector_Generic:Conn_01x06
- renumbered C8 to C10, C1 to C11, C7 to C12, C6 to C13, C9 to C14, C10 to C15, C11 to C16, C12 to C17, C13 to C18, C14 to C19, C15 to C20, C16 to C21, C17 to C22, C20 to C3, C21 to C4, C4 to C5, C5 to C6, C22 to C7, C2 to C8, C3 to C9, J1 to J3, R4 to R1, R5 to R2, R7 to R3, R1 to R4, R8 to R5, R2 to R7, R3 to R8, U4 to U2, U2 to U3, U1 to U4
Connections:
- net +3V3: now also J11.3 (Pin_3), J11.4 (Pin_4)
- net GND: now also J11.5 (Pin_5), J11.6 (Pin_6)
- net CAN_CS: now reaches U4.13 (GPIO9)
- net I2C1_SDA: now reaches U4.14 (GPIO10)
- net I2C1_SCL: now reaches U4.15 (GPIO11)
- net I2C0_SDA: now reaches U4.16 (GPIO12)
- net I2C0_SCL: now reaches U4.17 (GPIO13)
- net at U4.18 (GPIO14): now also J10.1 (Pin_1)
- net at U4.19 (GPIO15): now also J10.2 (Pin_2)
- net Buzzer: now reaches U4.2 (GPIO0)
- net at U4.27 (GPIO16): now also J10.3 (Pin_3)
- net at U4.28 (GPIO17): now also J10.4 (Pin_4)
- net at U4.29 (GPIO18): now also J10.5 (Pin_5)
- net at U4.31 (GPIO19): now also J10.6 (Pin_6)
- net at U4.32 (GPIO20): now also J10.7 (Pin_7)
- net at U4.33 (GPIO21): now also J10.8 (Pin_8)
- net at U4.34 (GPIO22): now also J10.9 (Pin_9)
- net at U4.35 (GPIO23): now also J10.10 (Pin_10)
- net at U4.36 (GPIO24): now also J10.11 (Pin_11)
- net at U4.37 (GPIO25): now also J10.12 (Pin_12)
- net CAN_SCK: now reaches U4.4 (GPIO2)
- net CAN_MOSI: now reaches U4.5 (GPIO3)
- net CAN_MISO: now reaches U4.7 (GPIO4)
- net CAN_INT: now reaches U4.8 (GPIO5)
- net VBUS renamed +5V
- net +5V: now also J11.1 (Pin_1), J11.2 (Pin_2)
- no-connect marks 3 -> 8

Commit message: 2026/02/12/1628
Parts:
- removed C3: 100n, Capacitor_SMD:C_0402_1005Metric, symbol Device:C
- removed U2: W25Q128JVS, Package_SO:SOIC-8_5.23x5.23mm_P1.27mm, symbol Memory_Flash:W25Q128JVS
- added C5: 100n, Capacitor_SMD:C_0402_1005Metric, symbol Device:C
- added D5: D, Diode_SMD:D_SMA, symbol Device:D
- added IC1: W25Q128JVSIQTR, rp2350:SOIC127P790X216-8N, symbol W25Q128JVSIQTR:W25Q128JVSIQTR
- C10, C11, C12, C13, C14, C15, C16, C17, C18, C19, C20, C21, C22: footprint (none) -> Capacitor_SMD:C_0402_1005Metric
- C4: renamed from C5; footprint (none) -> Capacitor_SMD:C_0805_2012Metric
- C6: footprint (none) -> Capacitor_SMD:C_0805_2012Metric
- C8, C9: footprint (none) -> RP2350_60QFN_minimal:C_0402_1005Metric_small_pads
- D2: renamed from D1; footprint (none) -> Diode_SMD:D_SMA
- D3: renamed from D2; footprint (none) -> Diode_SMD:D_SMA
- D4: renamed from D3; footprint (none) -> Diode_SMD:D_SMA
- J10: footprint (none) -> Connector_PinHeader_2.54mm:PinHeader_1x12_P2.54mm_Vertical
- J9: renamed from J11; footprint (none) -> Connector_PinHeader_2.54mm:PinHeader_1x06_P2.54mm_Vertical
- L1: footprint (none) -> RP2350_60QFN_minimal:L_pol_2016
- R1: value 10k -> 0; footprint Capacitor_SMD:C_0402_1005Metric -> Resistor_SMD:R_0402_1005Metric
- R2: value 0 -> 10k; footprint Capacitor_SMD:C_0402_1005Metric -> Resistor_SMD:R_0402_1005Metric
- R3, R6: footprint Capacitor_SMD:C_0402_1005Metric -> Resistor_SMD:R_0402_1005Metric
- R4, R5, R7, R8: footprint (none) -> Resistor_SMD:R_0402_1005Metric
- SW2: footprint (none) -> Button_Switch_SMD:SW_Push_1P1T_NO_Vertical_Wuerth_434133025816
- Y1: footprint SamacSys_Parts:ABM8272T3 -> Crystal:Crystal_SMD_3225-4Pin_3.2x2.5mm
- renumbered C4 to C3, J3 to J8, U3 to U2, U4 to U3
Connections:
- net +3V3: now also R2.2, C5.2, IC1.8 (VCC); no longer R1.2
- net +5V: now also D5.1 (K); no longer D3.1 (K), D4.1 (K), J9.1 (Pin_1), J9.2 (Pin_2)
- net Buzzer: now also U3.3 (GPIO1); no longer U3.2 (GPIO0)
- net GND: now also C5.1, IC1.4 (GND)
- net GPIO0: now also U3.2 (GPIO0), IC1.1 (~{CS})
- net QSPI_SCLK: now also IC1.6 (CLK)
- net QSPI_SD0: now also IC1.5 (DI_(IO0))
- net QSPI_SD1: now also IC1.2 (DO_(IO1))
- net QSPI_SD2: now also IC1.3 (~{WP_(IO2)})
- net QSPI_SD3: now also IC1.7 (~{HOLD_OR_}RESET_(IO3))
- net QSPI_SS: now also R1.2; no longer R2.2
- new net VBUS: D3.1 (K), D4.1 (K), D5.2 (A), J9.1 (Pin_1), J9.2 (Pin_2)
- no-connect marks 8 -> 7
