File: pilot/rp2350a.kicad_sch (KiCad schematic)
At the start: 42 parts, among them IC1 W25Q128JVSIQTR, J10 Conn_01x10, J8 USB_B_Micro, J9 Conn_01x06, SW1 SW_Push, SW2 SW_Push, U2 NCP1117-3.3_SOT223, U3 RP2350_60QFN, Y1 ABM8-272-T3

Commit message: 20261001
Parts:
- removed J8: USB_B_Micro, Connector_USB:USB_Micro-B_Amphenol_10103594-0001LF_Horizontal, symbol Connector:USB_B_Micro
- added J8: ZX62M-B-5P, rp2350:ZX62MB5P, symbol ZX62M-B-5P:ZX62M-B-5P
- renumbered R14 to R2, R2 to R3, R3 to R4, R4 to R5, R5 to R6, R6 to R7, R7 to R8, R8 to R9
Connections:
- net GND: now also J8.5, J8.MP1, J8.MP2, J8.MP3, J8.MP4, J8.MP5, J8.MP6
- net USB_D+: now also J8.3
- net USB_D-: now also J8.2
- net at D2.2 (A): now also J8.1
