File: pilot/untitled.kicad_sch (KiCad schematic)
At the start: 6 parts, among them Q1 2SC3325-Y,LF, SW3 SW_SPDT

Commit message: 2026/02/12/1628
Parts:
- LS1: footprint PKB24SPCH3601B0 -> rp2350:PKB24SPCH3601B0
- Q1: footprint 2SC3325YLF -> rp2350:2SC3325YLF
Changed lines of the file:
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@@
 		(dnp no)
 		(fields_autoplaced yes)
-		(property "Reference" "#PWR047"
+		(property "Reference" "#PWR063"
 			(at 133.35 168.91 0)
 			(effects
@@
 			(project "pilot"
 				(path "/6e01a02a-937c-45ab-a43c-49a8d1056ac9/dcfc96e1-e56d-42c9-b294-33f4cac85d9a"
-					(reference "#PWR047")
+					(reference "#PWR063")
 					(unit 1)
 				)
@@
 		(dnp no)
 		(fields_autoplaced yes)
-		(property "Reference" "#PWR045"
+		(property "Reference" "#PWR061"
 			(at 110.49 63.5 0)
 			(effects
@@
 			(project "pilot"
 				(path "/6e01a02a-937c-45ab-a43c-49a8d1056ac9/dcfc96e1-e56d-42c9-b294-33f4cac85d9a"
-					(reference "#PWR045")
+					(reference "#PWR061")
 					(unit 1)
 				)
@@
 		(dnp no)
 		(fields_autoplaced yes)
-		(property "Reference" "#PWR048"
+		(property "Reference" "#PWR064"
 			(at 144.78 92.71 0)
 			(effects
@@
 			(project "pilot"
 				(path "/6e01a02a-937c-45ab-a43c-49a8d1056ac9/dcfc96e1-e56d-42c9-b294-33f4cac85d9a"
-					(reference "#PWR048")
+					(reference "#PWR064")
 					(unit 1)
 				)
@@
 		(dnp no)
 		(fields_autoplaced yes)
-		(property "Reference" "#PWR046"
+		(property "Reference" "#PWR062"
 			(at 130.81 49.53 0)
 			(effects
@@
 			(project ""
 				(path "/6e01a02a-937c-45ab-a43c-49a8d1056ac9/dcfc96e1-e56d-42c9-b294-33f4cac85d9a"
-					(reference "#PWR046")
+					(reference "#PWR062")
 					(unit 1)
 				)
@@
 			)
 		)
-		(property "Footprint" "2SC3325YLF"
+		(property "Footprint" "rp2350:2SC3325YLF"
 			(at 137.16 232.08 0)
 			(effects
@@
 			)
 		)
-		(property "Footprint" "PKB24SPCH3601B0"
+		(property "Footprint" "rp2350:PKB24SPCH3601B0"
 			(at 142.24 180.01 0)
 			(effects
