File: pilot/untitled.kicad_sch (KiCad schematic)
At the start: 6 parts, among them Q1 2SC3325-Y,LF, SW3 SW_SPDT

Commit message: 20261001
Parts:
- renumbered R12 to R13, R13 to R14
Changed lines of the file:
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@@
 		(dnp no)
 		(fields_autoplaced yes)
-		(property "Reference" "R13"
+		(property "Reference" "R14"
 			(at 133.35 48.2599 0)
 			(effects
@@
 			(project "pilot"
 				(path "/6e01a02a-937c-45ab-a43c-49a8d1056ac9/dcfc96e1-e56d-42c9-b294-33f4cac85d9a"
-					(reference "R13")
+					(reference "R14")
 					(unit 1)
 				)
@@
 		(dnp no)
 		(fields_autoplaced yes)
-		(property "Reference" "R12"
+		(property "Reference" "R13"
 			(at 110.49 124.46 90)
 			(effects
@@
 			(project "pilot"
 				(path "/6e01a02a-937c-45ab-a43c-49a8d1056ac9/dcfc96e1-e56d-42c9-b294-33f4cac85d9a"
-					(reference "R12")
+					(reference "R13")
 					(unit 1)
 				)
