File: pilot/_autosave-rp2350a.kicad_sch (KiCad schematic)
At the start: 42 parts, among them IC1 W25Q128JVSIQTR, J10 Conn_01x12, J8 USB_B_Micro, J9 Conn_01x06, SW1 SW_Push, SW2 SW_Push, U2 NCP1117-3.3_SOT223, U3 RP2350_60QFN, Y1 ABM8-272-T3

Commit message: 2026/02/15
Parts:
- removed J10: Conn_01x12, Connector_PinHeader_2.54mm:PinHeader_1x12_P2.54mm_Vertical, symbol Connector_Generic:Conn_01x12
- added J10: Conn_01x10, Connector_PinHeader_2.54mm:PinHeader_1x10_P2.54mm_Vertical, symbol Connector_Generic:Conn_01x10
Connections:
- net Buzzer: now also U3.18 (GPIO14); no longer U3.3 (GPIO1)
- net at U3.27 (GPIO16): now also J10.1 (Pin_1)
- net at U3.28 (GPIO17): now also J10.2 (Pin_2)
- net at U3.29 (GPIO18): now also J10.3 (Pin_3)
- net at U3.31 (GPIO19): now also J10.4 (Pin_4)
- net at U3.32 (GPIO20): now also J10.5 (Pin_5)
- net at U3.33 (GPIO21): now also J10.6 (Pin_6)
- net at U3.34 (GPIO22): now also J10.7 (Pin_7)
- net at U3.35 (GPIO23): now also J10.8 (Pin_8)
- net at U3.36 (GPIO24): now also J10.9 (Pin_9)
- net at U3.37 (GPIO25): now also J10.10 (Pin_10)
- no-connect marks 7 -> 9
Changed lines of the file:
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@@
 	)
 	(no_connect
+		(at 246.38 158.75)
+	)
+	(no_connect
 		(at 182.88 223.52)
 	)
@@
 	)
 	(no_connect
+		(at 246.38 194.31)
+	)
+	(no_connect
 		(at 46.99 53.34)
 	)
@@
 	(wire
 		(pts
-			(xy 246.38 194.31) (xy 261.62 194.31)
-		)
-		(stroke
-			(width 0)
-			(type default)
-		)
-	)
-	(wire
-		(pts
 			(xy 36.83 58.42) (xy 36.83 60.96)
 		)
@@
 	(wire
 		(pts
-			(xy 246.38 191.77) (xy 261.62 191.77)
-		)
-		(stroke
-			(width 0)
-			(type default)
-		)
-	)
-	(wire
-		(pts
 			(xy 81.28 116.84) (xy 81.28 121.92)
 		)
@@
 	(hierarchical_label "Buzzer"
 		(shape input)
-		(at 246.38 158.75 0)
+		(at 246.38 191.77 0)
 		(effects
 			(font
@@
 	)
 	(symbol
+		(lib_id "Connector_Generic:Conn_01x10")
+		(at 266.7 207.01 0)
+		(unit 1)
+		(exclude_from_sim no)
+		(in_bom yes)
+		(on_board yes)
+		(dnp no)
+		(fields_autoplaced yes)
+		(property "Reference" "J10"
+			(at 269.24 207.0099 0)
+			(effects
+				(font
+					(size 1.27 1.27)
+				)
+				(justify left)
+			)
+		)
+		(property "Value" "Conn_01x10"
+			(at 269.24 209.5499 0)
+			(effects
+				(font
+					(size 1.27 1.27)
+				)
+				(justify left)
+			)
+		)
+		(property "Footprint" "Connector_PinHeader_2.54mm:PinHeader_1x10_P2.54mm_Vertical"
+			(at 266.7 207.01 0)
+			(effects
+				(font
+					(size 1.27 1.27)
+				)
+				(hide yes)
+			)
+		)
+		(property "Datasheet" "~"
+			(at 266.7 207.01 0)
+			(effects
+				(font
+					(size 1.27 1.27)
+				)
+				(hide yes)
+			)
+		)
+		(property "Description" "Generic connector, single row, 01x10, script generated (kicad-library-utils/schlib/autogen/connector/)"
+			(at 266.7 207.01 0)
+			(effects
+				(font
+					(size 1.27 1.27)
+				)
+				(hide yes)
+			)
+		)
+		(pin "1"
+		)
+		(pin "4"
+		)
+		(pin "9"
+		)
+		(pin "3"
+		)
+		(pin "2"
+		)
+		(pin "8"
+		)
+		(pin "6"
+		)
+		(pin "5"
+		)
+		(pin "7"
+		)
+		(pin "10"
+		)
+		(instances
+			(project ""
+				(path "/6e01a02a-937c-45ab-a43c-49a8d1056ac9/f8b94c15-0f98-420c-a532-2fade8bd7070"
+					(reference "J10")
+					(unit 1)
+				)
+			)
+		)
+	)
+	(symbol
 		(lib_id "power:GND")
 		(at 330.2 86.36 0)
@@
 					(unit 1)
 				)
-			)
-		)
-	)
-	(symbol
-		(lib_id "Connector_Generic:Conn_01x12")
-		(at 266.7 204.47 0)
-		(unit 1)
-		(exclude_from_sim no)
-		(in_bom yes)
-		(on_board yes)
-		(dnp no)
-		(fields_autoplaced yes)
-		(property "Reference" "J10"
-			(at 269.24 204.4699 0)
-			(effects
-				(font
-					(size 1.27 1.27)
-				)
-				(justify left)
-			)
-		)
-		(property "Value" "Conn_01x12"
-			(at 269.24 207.0099 0)
-			(effects
-				(font
-					(size 1.27 1.27)
-				)
-				(justify left)
-			)
-		)
-		(property "Footprint" "Connector_PinHeader_2.54mm:PinHeader_1x12_P2.54mm_Vertical"
-			(at 266.7 204.47 0)
-			(effects
-				(font
-					(size 1.27 1.27)
-				)
-				(hide yes)
-			)
-		)
-		(property "Datasheet" "~"
-			(at 266.7 204.47 0)
-			(effects
-				(font
-					(size 1.27 1.27)
-				)
-				(hide yes)
-			)
-		)
-		(property "Description" "Generic connector, single row, 01x12, script generated (kicad-library-utils/schlib/autogen/connector/)"
-			(at 266.7 204.47 0)
-			(effects
-				(font
-					(size 1.27 1.27)
-				)
-				(hide yes)
-			)
-		)
-		(pin "1"
-		)
-		(pin "2"
-		)
-		(pin "4"
-		)
-		(pin "3"
-		)
-		(pin "5"
-		)
-		(pin "6"
-		)
-		(pin "11"
-		)
-		(pin "9"
-		)
-		(pin "8"
-		)
-		(pin "10"
-		)
-		(pin "12"
-		)
-		(pin "7"
-		)
-		(instances
-			(project ""
-				(path "/6e01a02a-937c-45ab-a43c-49a8d1056ac9/f8b94c15-0f98-420c-a532-2fade8bd7070"
-					(reference "J10")
-					(unit 1)
-				)
