File: pilot/pilot.kicad_pcb (KiCad board)
At the start: 2 copper layers, 71 parts, among them IC1 W25Q128JVSIQTR, IC2 TJA1050T, J1 RJ45_Shielded, J10 Conn_01x12, J11 Conn_01x02, J2 Conn_01x03, J3 Conn_01x03, J4 Conn_01x03, J5 Conn_01x05, J6 Conn_01x04, J7 電源入力, J9 Conn_01x06, Q1 2SC3325-Y,LF, SW1 SW_Push, SW2 SW_Push, SW3 SW_SPDT, U1 NCP1117-5.0_SOT223, U2 NCP1117-3.3_SOT223, U3 RP2350_60QFN, U4 MCP2515-xSO, Y1 ABM8-272-T3, Y2 ABLS-8.000MHZ-12-B-4-Y-T

Commit message: 2026/02/12/1907
Routing:
- net +1V1: track 16.9 -> 31.0 mm, vias 5 -> 9
- net +3V3: track 16.6 -> 24.9 mm
- added copper zone on F.Cu, net +3V3

Commit message: 2026/02/15
Parts:
- removed D5: D, Diode_SMD:D_SMA
- added J8: USB_B_Micro, Connector_USB:USB_Micro-B_Amphenol_10103594-0001LF_Horizontal, F.Cu at (158.4, 55.7)
- added R14: DNF, Capacitor_SMD:C_0402_1005Metric, F.Cu at (147.8, 74.8)
- J10: value Conn_01x12 -> Conn_01x10; footprint Connector_PinHeader_2.54mm:PinHeader_1x12_P2.54mm_Vertical -> Connector_PinHeader_2.54mm:PinHeader_1x10_P2.54mm_Vertical
- J7: footprint Connector_JST:JST_VH_B2P-VH-B_1x02_P3.96mm_Vertical -> Connector_JST:JST_VH_B2P-VH-FB-B_1x02_P3.96mm_Vertical
- R2: value 10k -> DNF
- moved J3 159.8 mm to (180.2, 105.7)
- moved J2 159.3 mm to (180.1, 96.3)
- moved J4 154.0 mm to (180.2, 88.1)
- moved J7 134.9 mm to (175.7, 60.8), turned to 180 degrees
- moved LS1 132.8 mm to (165.2, 131.1)
- moved C2 129.5 mm to (180.2, 69.5), turned to 90 degrees
- moved U1 127.9 mm to (174.2, 70.4)
- moved J6 119.8 mm to (144.4, 103.6), turned to 180 degrees
- moved J10 118.4 mm to (172.9, 113.8), turned to 180 degrees
- moved C1 118.1 mm to (168.6, 70.5), turned to 90 degrees
- moved C28 117.2 mm to (185.2, 115.9)
- moved R13 115.0 mm to (180.4, 114.9), turned to -90 degrees
- moved C26 114.9 mm to (141.3, 81.6), turned to 180 degrees
- moved R10 114.8 mm to (141.3, 83.5)
- moved R9 114.8 mm to (141.1, 77.4), turned to 180 degrees
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Connections:
- D3 pad 1: VBUS -> +5V
- D4 pad 1: VBUS -> +5V
- IC1 pad 1: /rp2350a/GPIO0 -> Net-(IC1-~{CS})
- J1 pad 1: /CAN_L -> /CAN_H
- J1 pad 2: /CAN_H -> /CAN_L
- J9 pad 1: VBUS -> +5V
- J9 pad 2: VBUS -> +5V
- R1 pad 1: /rp2350a/GPIO0 -> Net-(IC1-~{CS})
- R2 pad 1: /rp2350a/GPIO0 -> Net-(IC1-~{CS})
- U3 pad 18: Net-(J10-Pin_1) -> /Buzzer
- U3 pad 19: Net-(J10-Pin_2) -> unconnected-(U3-GPIO15-Pad19)
- U3 pad 27: Net-(J10-Pin_3) -> Net-(J10-Pin_1)
- U3 pad 28: Net-(J10-Pin_4) -> Net-(J10-Pin_2)
- U3 pad 29: Net-(J10-Pin_5) -> Net-(J10-Pin_3)
- U3 pad 3: /Buzzer -> unconnected-(U3-GPIO1-Pad3)
- U3 pad 31: Net-(J10-Pin_6) -> Net-(J10-Pin_4)
- U3 pad 32: Net-(J10-Pin_7) -> Net-(J10-Pin_5)
- U3 pad 33: Net-(J10-Pin_8) -> Net-(J10-Pin_6)
- U3 pad 34: Net-(J10-Pin_9) -> Net-(J10-Pin_7)
- U3 pad 35: Net-(J10-Pin_10) -> Net-(J10-Pin_8)
- U3 pad 36: Net-(J10-Pin_11) -> Net-(J10-Pin_9)
- U3 pad 37: Net-(J10-Pin_12) -> Net-(J10-Pin_10)
Routing:
- net +5V: track 0.00 -> 148.6 mm, vias 0 -> 7
- net +3V3: track 24.9 -> 159.1 mm, vias 0 -> 4
- net GND: track 9.59 -> 100.3 mm, vias 10 -> 40
- net /CAN_L: track 0.00 -> 32.6 mm, vias 0 -> 1
- net /LAD_ADC: track 0.00 -> 32.4 mm
- net /Buzzer: track 0.00 -> 28.3 mm
- net /rp2350a/GPIO0: track 0.00 -> 26.8 mm, vias 0 -> 2
- net /rp2350a/USB_D+: track 0.00 -> 25.2 mm
- net /rp2350a/USB_D-: track 0.00 -> 25.0 mm
- net /rp2350a/QSPI_SS: track 0.00 -> 24.9 mm
- net /CAN_H: track 0.00 -> 24.7 mm
- net Net-(J10-Pin_1): track 0.00 -> 24.6 mm
- net /ELE_ADC: track 0.00 -> 24.5 mm
- net /SIM_SDA: track 0.00 -> 23.0 mm
- net /SIM_SCL: track 0.00 -> 22.2 mm
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- added copper zone on F.Cu, net +5V
- added copper zone on B.Cu, net GND
Other:
- board outline added: 72.3 x 98.3 mm

Commit message: 2026/02/24/1620
Changed lines of the file:
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@@
-	)
-	(segment
-		(start 147.77 74.32)
-		(end 147.77 73.05)
-		(width 0.15)
-		(layer "F.Cu")
-		(net 5)
 	)
 	(segment
@@
 	)
 	(segment
+		(start 147.77 74.32)
+		(end 147.77 73.54)
+		(width 0.15)
+		(layer "F.Cu")
+		(net 5)
+	)
+	(segment
+		(start 147.77 73.54)
+		(end 147.47 73.24)
+		(width 0.15)
+		(layer "F.Cu")
+		(net 5)
+	)
+	(segment
 		(start 151.57 87.01)
 		(end 152.86 88.3)
@@
 	)
 	(via
-		(at 147.77 73.05)
+		(at 147.47 73.24)
 		(size 0.6)
 		(drill 0.35)
@@
 	)
 	(segment
+		(start 149.18 84.65)
+		(end 151.54 87.01)
+		(width 0.15)
+		(layer "B.Cu")
+		(net 5)
+	)
+	(segment
+		(start 144.33 82.51)
+		(end 146.47 84.65)
+		(width 0.15)
+		(layer "B.Cu")
+		(net 5)
+	)
+	(segment
+		(start 144.33 75.55)
+		(end 144.33 82.51)
+		(width 0.15)
+		(layer "B.Cu")
+		(net 5)
+	)
+	(segment
+		(start 146.83 73.05)
+		(end 144.33 75.55)
+		(width 0.15)
+		(layer "B.Cu")
+		(net 5)
+	)
+	(segment
 		(start 151.54 87.01)
+		(end 151.57 87.01)
+		(width 0.15)
+		(layer "B.Cu")
+		(net 5)
+	)
+	(segment
+		(start 147.28 73.05)
+		(end 146.83 73.05)
+		(width 0.15)
+		(layer "B.Cu")
+		(net 5)
+	)
+	(segment
+		(start 146.47 84.65)
 		(end 149.18 84.65)
 		(width 0.15)
@@
 	)
 	(segment
-		(start 144.33 75.55)
-		(end 146.83 73.05)
-		(width 0.15)
-		(layer "B.Cu")
-		(net 5)
-	)
-	(segment
-		(start 151.57 87.01)
-		(end 151.54 87.01)
-		(width 0.15)
-		(layer "B.Cu")
-		(net 5)
-	)
-	(segment
-		(start 146.47 84.65)
-		(end 144.33 82.51)
-		(width 0.15)
-		(layer "B.Cu")
-		(net 5)
-	)
-	(segment
-		(start 146.83 73.05)
-		(end 147.77 73.05)
-		(width 0.15)
-		(layer "B.Cu")
-		(net 5)
-	)
-	(segment
-		(start 144.33 82.51)
-		(end 144.33 75.55)
-		(width 0.15)
-		(layer "B.Cu")
-		(net 5)
-	)
-	(segment
-		(start 149.18 84.65)
-		(end 146.47 84.65)
+		(start 147.47 73.24)
+		(end 147.28 73.05)
 		(width 0.15)
 		(layer "B.Cu")
@@
 		(start 169.3275 72.7475)
 		(end 171.08 72.7475)
-		(width 0.15)
+		(width 1)
 		(layer "F.Cu")
 		(net 10)
@@
 		(start 168.09 71.52)
 		(end 169.26 72.69)
-		(width 0.15)
-		(layer "F.Cu")
-		(net 10)
-	)
-	(segment
-		(start 169.27 72.69)
-		(end 169.3275 72.7475)
-		(width 0.15)
+		(width 1)
 		(layer "F.Cu")
 		(net 10)
@@
 				(xy 120.53 116.09) (xy 133.03 115.64) (xy 133.98 97.66) (xy 147.75 96.95) (xy 147.89 84.43) (xy 153.75 84.72)
 				(xy 154.19 93.81) (xy 155.01 95.53) (xy 165.12 95.24) (xy 170.27 89.5) (xy 177.14 89.33) (xy 177.08 110.35)
-				(xy 181.69 112.15) (xy 184.13 113.78) (xy 184.09 148.71) (xy 120.39 146.23)
+				(xy 181.69 112.15) (xy 184.13 113.78) (xy 184.09 148.71) (xy 121.82 148.56)
 			)
 		)
