File: pilot/pilot.kicad_pcb (KiCad board)
At the start: 2 copper layers, 72.3 x 98.3 mm, 72 parts, among them IC1 W25Q128JVSIQTR, IC2 TJA1050T, J1 RJ45_Shielded, J10 Conn_01x10, J11 Conn_01x02, J2 Conn_01x03, J3 Conn_01x03, J4 Conn_01x03, J5 Conn_01x05, J6 Conn_01x04, J7 電源入力, J8 USB_B_Micro, J9 Conn_01x06, Q1 2SC3325-Y,LF, SW1 SW_Push, SW2 SW_Push, SW3 SW_SPDT, U1 NCP1117-5.0_SOT223, U2 NCP1117-3.3_SOT223, U3 RP2350_60QFN, U4 MCP2515-xSO, Y1 ABM8-272-T3, Y2 ABLS-8.000MHZ-12-B-4-Y-T

Commit message: 20261001
Parts:
- removed the R14 at (147.8, 74.8)
- added R2: DNF, Capacitor_SMD:C_0402_1005Metric, F.Cu at (149.3, 74.3)
- D5: renamed from D6; footprint Diode_SMD:D_SMA -> LED_SMD:LED_0603_1608Metric
- J8: value USB_B_Micro -> ZX62M-B-5P; footprint Connector_USB:USB_Micro-B_Amphenol_10103594-0001LF_Horizontal -> rp2350:ZX62MB5P
- moved R3 1.49 mm to (150.9, 74.8)
- moved J8 0.83 mm to (158.6, 54.9)
- renumbered R9 to R10, R10 to R11, R11 to R12, R12 to R13, R13 to R14, R2 to R3, R3 to R4, R4 to R5, R5 to R6, R6 to R7, R7 to R8, R8 to R9
Routing:
- net GND: track 100.3 -> 109.7 mm, vias 40 -> 31
- net Net-(IC1-~{CS}): track 5.32 -> 7.85 mm
- net /rp2350a/USB_D-: track 25.0 -> 23.0 mm
- net /rp2350a/USB_D+: track 25.2 -> 23.3 mm
- net Net-(D2-A): track 11.2 -> 9.30 mm
- net +3V3: track 159.1 -> 157.6 mm
- net Net-(D5-A): track 5.98 -> 7.20 mm
- net /rp2350a/GPIO0: track 26.5 -> 27.6 mm
Other:
- outline, holes or cut-outs redrawn
