File: logger/logger/bme280.kicad_sch (KiCad schematic)
At the start: 4 parts, among them U6 BME280

Commit message: 2026/02/24/1620
Parts:
- C29, C30: footprint Capacitor_SMD:C_0805_2012Metric -> Capacitor_SMD:C_0402_1005Metric
Connections:
- net +3V3: now also C30.2; no longer C30.1
- net GND: now also C30.1; no longer C30.2
