File: logger/logger/logger.kicad_sch (KiCad schematic)
At the start: 9 parts, among them J1 RJ45_Shielded, J10 Conn_01x06, J2 電源入力, J3 Conn_01x04, J8 Conn_01x03, J9 Conn_01x04, U1 NCP1117-5.0_SOT223

Commit message: 2026/02/24/1620
Parts:
- added R21, R22: 2.2k, Resistor_SMD:R_0402_1005Metric, symbol Device:R
- added R23, R24: 4.7k, Resistor_SMD:R_0402_1005Metric, symbol Device:R
Connections:
- net +3.3V is gone; now on net +3V3: J8.2 (Pin_2)
- net +3V3: now also R21.1, R22.1, R23.1, R24.1
- net I2C0_SCL: now also R22.2
- net I2C0_SDA: now also R21.2
- net I2C1_SCL: now also R24.2
- net I2C1_SDA: now also R23.2
