File: logger/logger/rp2350a.kicad_sch (KiCad schematic)
At the start: 42 parts, among them IC1 W25Q128JVSIQTR, J10 Conn_01x10, J8 USB_B_Micro, J9 Conn_01x06, SW1 SW_Push, SW2 SW_Push, U2 NCP1117-3.3_SOT223, U3 RP2350_60QFN, Y1 ABM8-272-T3

Commit message: 2026/02/23
Parts:
- removed J10: Conn_01x10, Connector_PinHeader_2.54mm:PinHeader_1x10_P2.54mm_Vertical, symbol Connector_Generic:Conn_01x10
- removed R14: DNF, Capacitor_SMD:C_0402_1005Metric, symbol Device:R
- added D6: D, Diode_SMD:D_SMA, symbol Device:D
- added R2: DNF, Resistor_SMD:R_0402_1005Metric, symbol Device:R
- IC1: footprint rp2350:SOIC127P790X216-8N -> footprint:SOIC127P790X216-8N
- renumbered D2 to D1, D3 to D2, D4 to D3, J8 to J4, J9 to J5, R2 to R3, R3 to R4, R4 to R5, R5 to R6, R6 to R7, R7 to R8, R8 to R9
Connections:
- net Buzzer is gone; now on net I2C1_SDA: U3.18 (GPIO14)
- net +5V: now also D6.1 (K); no longer D2.1 (K), D3.1 (K), J5.1 (Pin_1), J5.2 (Pin_2)
- net CAN_CS: now also U3.28 (GPIO17); no longer U3.13 (GPIO9)
- net CAN_INT: now also U3.32 (GPIO20); no longer U3.8 (GPIO5)
- net CAN_MISO: now also U3.27 (GPIO16); no longer U3.7 (GPIO4)
- net CAN_MOSI: now also U3.31 (GPIO19); no longer U3.5 (GPIO3)
- net CAN_SCK: now also U3.29 (GPIO18); no longer U3.4 (GPIO2)
- net GPIO0: now also R2.1
- net I2C0_SCL: now also U3.13 (GPIO9); no longer U3.17 (GPIO13)
- net I2C0_SDA: now also U3.12 (GPIO8); no longer U3.16 (GPIO12)
- net I2C1_SCL: now also U3.19 (GPIO15); no longer U3.15 (GPIO11)
- net I2C1_SDA: no longer U3.14 (GPIO10)
- net SD_CS: now reaches U3.3 (GPIO1)
- net at IC1.1 (~{CS}), R1.1, R3.1: now also R2.2
- net ELE_ADC: no longer names the net of U3.41 (GPIO27_ADC1)
- net LAD_ADC renamed ADC0
- net SPARE_ADC: no longer names the net of U3.42 (GPIO28_ADC2)
- new net SD_MISO: U3.7 (GPIO4)
- new net SD_MOSI: U3.5 (GPIO3)
- new net SD_SCK: U3.4 (GPIO2)
- new net VBUS: D2.1 (K), D3.1 (K), D6.2 (A), J5.1 (Pin_1), J5.2 (Pin_2)
- no-connect marks 9 -> 18
Other:
- moved on the sheet: C10, C11, C12, C13, C14, C15, C16, C17, C18, C19, C20, C21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

Commit message: 2026/02/24/1620
Parts:
- removed D6: D, Diode_SMD:D_SMA, symbol Device:D
- removed J5: Conn_01x06, Connector_PinHeader_2.54mm:PinHeader_1x06_P2.54mm_Vertical, symbol Connector_Generic:Conn_01x06
Connections:
- net VBUS is gone; now on net +5V: D2.1 (K), D3.1 (K)
- net I2C0_SCL: now also U3.8 (GPIO5); no longer U3.13 (GPIO9)
- net I2C0_SDA: now also U3.7 (GPIO4); no longer U3.12 (GPIO8)
- net SD_CS: now also U3.13 (GPIO9); no longer U3.3 (GPIO1)
- net SD_MISO: now also U3.12 (GPIO8); no longer U3.7 (GPIO4)
- net SD_MOSI: now also U3.10 (GPIO7); no longer U3.5 (GPIO3)
- net SD_SCK: now also U3.9 (GPIO6); no longer U3.4 (GPIO2)
