File: logger/logger/logger.kicad_pcb (KiCad board)
At the start: 2 copper layers, 87 parts, among them IC1 W25Q128JVSIQTR, IC2 TJA1050T, IC3 BNO085, J1 RJ45_Shielded, J10 Conn_01x06, J2 電源入力, J3 Conn_01x04, J4 USB_B_Micro, J6 Conn_01x02, J7 DM3AT-SF-PEJM5_40_, J8 Conn_01x03, J9 Conn_01x04, SW1 SW_Push, SW2 SW_Push, U1 NCP1117-5.0_SOT223, U2 NCP1117-3.3_SOT223, U3 RP2350_60QFN, U4 MCP2515-xSO, U5 BMP581, U6 BME280, Y1 ABM8-272-T3, Y2 ABLS-8.000MHZ-12-B-4-Y-T, Y3 NX3215SA-32.768K-STD-MUA-8

Commit message: 2026/02/24/1820
Parts:
- moved C1 82.2 mm to (121.3, 78.6)
- moved C11 82.2 mm to (115.7, 83.5)
- moved C13 82.2 mm to (105.0, 87.6)
- moved C14 82.2 mm to (115.0, 93.5)
- moved C18 82.2 mm to (105.5, 84.5)
- moved C20 82.2 mm to (117.3, 85.1)
- moved C21 82.2 mm to (117.2, 86.3)
- moved C26 82.2 mm to (116.4, 109.7)
- moved C32 82.2 mm to (91.1, 85.4)
- moved C34 82.2 mm to (99.3, 97.9)
- moved C5 82.2 mm to (109.5, 96.3)
- moved C6 82.2 mm to (118.2, 81.9)
- moved C7 82.2 mm to (112.3, 98.8)
- moved IC3 82.2 mm to (97.9, 90.1)
- moved J3 82.2 mm to (99.9, 103.8)
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Routing:
- net GND: track 71.3 -> 130.9 mm, vias 31 -> 53
- net +3V3: track 314.3 -> 321.8 mm, vias 18 -> 19
- net Net-(U4-OSC1): track 7.42 -> 11.7 mm
- net Net-(U4-OSC2): track 9.41 -> 13.7 mm
- net Net-(J2-Pin_2): track 29.7 -> 31.0 mm
- added copper zone on F.Cu, net +5V
- added copper zone on B.Cu, net GND
- added copper zone on F.Cu, net GND
Other:
- board outline added: 74.2 x 69.4 mm
