File: logger/logger.kicad_pcb (KiCad board)
At the start: 2 copper layers, 74.2 x 69.4 mm, 87 parts, among them IC1 W25Q128JVSIQTR, IC2 TJA1050T, IC3 BNO085, J1 RJ45_Shielded, J10 Conn_01x06, J2 電源入力, J3 Conn_01x04, J4 USB_B_Micro, J6 Conn_01x02, J7 DM3AT-SF-PEJM5_40_, J8 Conn_01x03, J9 Conn_01x04, SW1 SW_Push, SW2 SW_Push, U1 NCP1117-5.0_SOT223, U2 NCP1117-3.3_SOT223, U3 RP2350_60QFN, U4 MCP2515-xSO, U5 BMP581, U6 BME280, Y1 ABM8-272-T3, Y2 ABLS-8.000MHZ-12-B-4-Y-T, Y3 NX3215SA-32.768K-STD-MUA-8

Commit message: 202603301205
Parts:
- added C36: 100n, Capacitor_SMD:C_0402_1005Metric, F.Cu at (105.0, 92.0)
Routing:
- net +3V3: track 321.8 -> 324.8 mm, vias 19 -> 18
- net GND: track 130.9 -> 131.1 mm, vias 53 -> 54
