File: logger/CAN.kicad_sch (KiCad schematic)
At the start: 14 parts, among them IC2 TJA1050T, J6 Conn_01x02, U4 MCP2515-xSO, Y2 ABLS-8.000MHZ-12-B-4-Y-T

Commit message: 20261001
Parts:
- D4: footprint Diode_SMD:D_SMA -> LED_SMD:LED_0603_1608Metric
Changed lines of the file:
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@@
 			)
 		)
-		(property "Footprint" "Diode_SMD:D_SMA"
+		(property "Footprint" "LED_SMD:LED_0603_1608Metric"
 			(at 104.14 71.12 0)
 			(effects
