File: logger/logger.kicad_sch (KiCad schematic)
At the start: 13 parts, among them J1 RJ45_Shielded, J10 Conn_01x06, J2 電源入力, J3 Conn_01x04, J8 Conn_01x03, J9 Conn_01x04, U1 NCP1117-5.0_SOT223

Commit message: 20261001
Other:
- moved on the sheet: J10, J9
Changed lines of the file:
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@@
-	)
-	(junction
-		(at 113.03 134.62)
-		(diameter 0)
-		(color 0 0 0 0)
 	)
 	(junction
@@
 	)
 	(label "CAN_MISO"
-		(at 146.05 182.88 180)
+		(at 63.5 193.04 180)
 		(effects
 			(font
@@
 	)
 	(label "CAN_CS"
-		(at 146.05 175.26 180)
+		(at 63.5 185.42 180)
 		(effects
 			(font
@@
 	)
 	(label "I2C1_SCL"
-		(at 146.05 157.48 180)
+		(at 63.5 167.64 180)
 		(effects
 			(font
@@
 	)
 	(label "CAN_SCK"
-		(at 146.05 177.8 180)
+		(at 63.5 187.96 180)
 		(effects
 			(font
@@
 	)
 	(label "CAN_MOSI"
-		(at 146.05 180.34 180)
+		(at 63.5 190.5 180)
 		(effects
 			(font
@@
 	)
 	(label "I2C1_SDA"
-		(at 146.05 160.02 180)
+		(at 63.5 170.18 180)
 		(effects
 			(font
@@
 	(symbol
 		(lib_id "Connector_Generic:Conn_01x06")
-		(at 151.13 175.26 0)
+		(at 68.58 185.42 0)
 		(unit 1)
 		(exclude_from_sim no)
@@
 		(fields_autoplaced yes)
 		(property "Reference" "J10"
-			(at 153.67 175.2599 0)
+			(at 71.12 185.4199 0)
 			(effects
 				(font
@@
 		)
 		(property "Value" "Conn_01x06"
-			(at 153.67 177.7999 0)
+			(at 71.12 187.9599 0)
 			(effects
 				(font
@@
 		)
 		(property "Footprint" "Connector_JST:JST_XH_B6B-XH-AM_1x06_P2.50mm_Vertical"
-			(at 151.13 175.26 0)
+			(at 68.58 185.42 0)
 			(effects
 				(font
@@
 		)
 		(property "Datasheet" "~"
-			(at 151.13 175.26 0)
+			(at 68.58 185.42 0)
 			(effects
 				(font
@@
 		)
 		(property "Description" "Generic connector, single row, 01x06, script generated (kicad-library-utils/schlib/autogen/connector/)"
-			(at 151.13 175.26 0)
+			(at 68.58 185.42 0)
 			(effects
 				(font
@@
 	(symbol
 		(lib_id "Connector_Generic:Conn_01x04")
-		(at 151.13 157.48 0)
+		(at 68.58 167.64 0)
 		(unit 1)
 		(exclude_from_sim no)
@@
 		(fields_autoplaced yes)
 		(property "Reference" "J9"
-			(at 153.67 157.4799 0)
+			(at 71.12 167.6399 0)
 			(effects
 				(font
@@
 		)
 		(property "Value" "Conn_01x04"
-			(at 153.67 160.0199 0)
+			(at 71.12 170.1799 0)
 			(effects
 				(font
@@
 		)
 		(property "Footprint" "Connector_JST:JST_XH_B4B-XH-AM_1x04_P2.50mm_Vertical"
-			(at 151.13 157.48 0)
+			(at 68.58 167.64 0)
 			(effects
 				(font
@@
 		)
 		(property "Datasheet" "~"
-			(at 151.13 157.48 0)
+			(at 68.58 167.64 0)
 			(effects
 				(font
@@
 		)
 		(property "Description" "Generic connector, single row, 01x04, script generated (kicad-library-utils/schlib/autogen/connector/)"
-			(at 151.13 157.48 0)
+			(at 68.58 167.64 0)
 			(effects
 				(font
@@
 	(symbol
 		(lib_id "power:GND")
-		(at 146.05 172.72 270)
+		(at 63.5 182.88 270)
 		(mirror x)
 		(unit 1)
@@
 		(dnp no)
 		(property "Reference" "#PWR087"
-			(at 139.7 172.72 0)
+			(at 57.15 182.88 0)
 			(effects
 				(font
@@
 		)
 		(property "Value" "GND"
-			(at 142.24 172.7199 90)
+			(at 59.69 182.8799 90)
 			(effects
 				(font
@@
 		)
 		(property "Footprint" ""
-			(at 146.05 172.72 0)
+			(at 63.5 182.88 0)
 			(effects
 				(font
@@
 		)
 		(property "Datasheet" ""
-			(at 146.05 172.72 0)
+			(at 63.5 182.88 0)
 			(effects
 				(font
@@
 		)
 		(property "Description" "Power symbol creates a global label with name \"GND\" , ground"
-			(at 146.05 172.72 0)
+			(at 63.5 182.88 0)
 			(effects
 				(font
@@
 	(symbol
 		(lib_id "power:+3V3")
-		(at 146.05 154.94 90)
+		(at 63.5 165.1 90)
 		(unit 1)
 		(exclude_from_sim no)
@@
 		(fields_autoplaced yes)
 		(property "Reference" "#PWR084"
-			(at 149.86 154.94 0)
+			(at 67.31 165.1 0)
 			(effects
 				(font
@@
 		)
 		(property "Value" "+3V3"
-			(at 142.24 154.9399 90)
+			(at 59.69 165.0999 90)
 			(effects
 				(font
@@
 		)
 		(property "Footprint" ""
-			(at 146.05 154.94 0)
+			(at 63.5 165.1 0)
 			(effects
 				(font
@@
 		)
 		(property "Datasheet" ""
-			(at 146.05 154.94 0)
+			(at 63.5 165.1 0)
 			(effects
 				(font
@@
 		)
 		(property "Description" "Power symbol creates a global label with name \"+3V3\""
-			(at 146.05 154.94 0)
+			(at 63.5 165.1 0)
 			(effects
 				(font
@@
 	(symbol
 		(lib_id "power:+3V3")
-		(at 146.05 170.18 90)
+		(at 63.5 180.34 90)
 		(unit 1)
 		(exclude_from_sim no)
@@
 		(fields_autoplaced yes)
 		(property "Reference" "#PWR086"
-			(at 149.86 170.18 0)
+			(at 67.31 180.34 0)
 			(effects
 				(font
@@
 		)
 		(property "Value" "+3V3"
-			(at 142.24 170.1799 90)
+			(at 59.69 180.3399 90)
 			(effects
 				(font
@@
 		)
 		(property "Footprint" ""
-			(at 146.05 170.18 0)
+			(at 63.5 180.34 0)
 			(effects
 				(font
@@
 		)
 		(property "Datasheet" ""
-			(at 146.05 170.18 0)
+			(at 63.5 180.34 0)
 			(effects
 				(font
@@
 		)
 		(property "Description" "Power symbol creates a global label with name \"+3V3\""
-			(at 146.05 170.18 0)
+			(at 63.5 180.34 0)
 			(effects
 				(font
@@
 	(symbol
 		(lib_id "power:GND")
-		(at 146.05 162.56 270)
+		(at 63.5 172.72 270)
 		(mirror x)
 		(unit 1)
@@
 		(dnp no)
 		(property "Reference" "#PWR085"
-			(at 139.7 162.56 0)
+			(at 57.15 172.72 0)
 			(effects
 				(font
@@
 		)
 		(property "Value" "GND"
-			(at 142.24 162.5599 90)
+			(at 59.69 172.7199 90)
 			(effects
 				(font
@@
 		)
 		(property "Footprint" ""
-			(at 146.05 162.56 0)
+			(at 63.5 172.72 0)
 			(effects
 				(font
@@
 		)
 		(property "Datasheet" ""
-			(at 146.05 162.56 0)
+			(at 63.5 172.72 0)
 			(effects
 				(font
@@
 		)
 		(property "Description" "Power symbol creates a global label with name \"GND\" , ground"
-			(at 146.05 162.56 0)
+			(at 63.5 172.72 0)
 			(effects
 				(font
@@
 					(unit 1)
 				)
-			)
-		)
-	)
-	(symbol
-		(lib_id "power:PWR_FLAG")
-		(at 113.03 134.62 0)
-		(unit 1)
-		(exclude_from_sim no)
-		(in_bom yes)
-		(on_board yes)
-		(dnp no)
-		(fields_autoplaced yes)
-		(property "Reference" "#FLG06"
-			(at 113.03 132.715 0)
-			(effects
-				(font
-					(size 1.27 1.27)
-				)
-				(hide yes)
-			)
-		)
-		(property "Value" "PWR_FLAG"
-			(at 113.03 129.54 0)
-			(effects
-				(font
-					(size 1.27 1.27)
-				)
-			)
-		)
-		(property "Footprint" ""
-			(at 113.03 134.62 0)
-			(effects
-				(font
-					(size 1.27 1.27)
-				)
-				(hide yes)
-			)
-		)
-		(property "Datasheet" "~"
-			(at 113.03 134.62 0)
-			(effects
-				(font
-					(size 1.27 1.27)
-				)
-				(hide yes)
-			)
-		)
-		(property "Description" "Special symbol for telling ERC where power comes from"
-			(at 113.03 134.62 0)
-			(effects
-				(font
-					(size 1.27 1.27)
-				)
-				(hide yes)
-			)
-		)
-		(pin "1"
-		)
-		(instances
-			(project ""
-				(path "/edd79af4-7743-4a3d-8195-b3e68f0873bc"
-					(reference "#FLG06")
-					(unit 1)
-				)
