File: logger/rp2350a.kicad_sch (KiCad schematic)
At the start: 41 parts, among them IC1 W25Q128JVSIQTR, J4 USB_B_Micro, SW1 SW_Push, SW2 SW_Push, U2 NCP1117-3.3_SOT223, U3 RP2350_60QFN, Y1 ABM8-272-T3

Commit message: 20261001
Parts:
- removed J4: USB_B_Micro, Connector_USB:USB_Micro-B_Amphenol_10103594-0001LF_Horizontal, symbol Connector:USB_B_Micro
- added J5: ZX62M-B-5P, footprint:ZX62MB5P, symbol ZX62M-B-5P:ZX62M-B-5P
Connections:
- net GND: now also J5.5, J5.MP1, J5.MP2, J5.MP3, J5.MP4, J5.MP5, J5.MP6
- net USB_D+: now also J5.3
- net USB_D-: now also J5.2
- net at D1.2 (A): now also J5.1
