File: pitot_tube/rp2350.kicad_sch (KiCad schematic)
At the start: 40 parts, among them IC1 W25Q128JVSIQTR, J4 USB_B_Micro, SW1 SW_Push, SW2 SW_Push, U2 NCP1117-3.3_SOT223, U3 RP2350_60QFN, Y1 ABM8-272-T3

Commit message: 202603301205
Parts:
- IC1: footprint footprint:SOIC127P790X216-8N -> footprints:SOIC127P790X216-8N
Connections:
- net SD_CS is gone; now on net CAN_CS: U3.13 (GPIO9)
- net CAN_CS: no longer U3.28 (GPIO17)
- net CAN_INT: now also U3.17 (GPIO13); no longer U3.32 (GPIO20)
- net CAN_MISO: now also U3.16 (GPIO12); no longer U3.27 (GPIO16)
- net CAN_MOSI: now also U3.15 (GPIO11); no longer U3.31 (GPIO19)
- net CAN_SCK: now also U3.14 (GPIO10); no longer U3.29 (GPIO18)
- net ADC0: no longer names the net of U3.40 (GPIO26_ADC0)
- net I2C0_SCL: no longer names the net of U3.8 (GPIO5)
- net I2C0_SDA: no longer names the net of U3.7 (GPIO4)
- net I2C1_SCL: no longer names the net of U3.19 (GPIO15)
- net I2C1_SDA: no longer names the net of U3.18 (GPIO14)
- net SD_MISO: no longer names the net of U3.12 (GPIO8)
- net SD_MOSI renamed SCL
- net SD_SCK renamed SDA
- no-connect marks 18 -> 25
Other:
- moved on the sheet: C10, C11, C12, C13, C14, C15, C16, C17, C18, C19, C20, C21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
