File: power/CAN.kicad_sch (KiCad schematic)
At the start: 12 parts, among them IC2 TJA1050T, J14 Conn_01x02, U2 MCP2515-xSO, Y2 ABLS-8.000MHZ-12-B-4-Y-T

Commit message: 2026/04/01
Parts:
- renumbered J14 to J13
Changed lines of the file:
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@@
 		(dnp no)
 		(fields_autoplaced yes)
-		(property "Reference" "#PWR062"
+		(property "Reference" "#PWR064"
 			(at 209.55 110.49 0)
 			(effects
@@
 			(project "power"
 				(path "/b905a668-e7ff-483f-a1a5-78bb0590864b/f3b54294-78cd-476f-bb66-930d59da1e95"
-					(reference "#PWR062")
+					(reference "#PWR064")
 					(unit 1)
 				)
@@
 		(dnp no)
 		(fields_autoplaced yes)
-		(property "Reference" "#PWR054"
+		(property "Reference" "#PWR056"
 			(at 153.67 143.51 0)
 			(effects
@@
 			(project "power"
 				(path "/b905a668-e7ff-483f-a1a5-78bb0590864b/f3b54294-78cd-476f-bb66-930d59da1e95"
-					(reference "#PWR054")
+					(reference "#PWR056")
 					(unit 1)
 				)
@@
 		(dnp no)
 		(fields_autoplaced yes)
-		(property "Reference" "#PWR059"
+		(property "Reference" "#PWR061"
 			(at 172.72 104.14 0)
 			(effects
@@
 			(project "power"
 				(path "/b905a668-e7ff-483f-a1a5-78bb0590864b/f3b54294-78cd-476f-bb66-930d59da1e95"
-					(reference "#PWR059")
+					(reference "#PWR061")
 					(unit 1)
 				)
@@
 		(dnp no)
 		(fields_autoplaced yes)
-		(property "Reference" "#PWR040"
+		(property "Reference" "#PWR042"
 			(at 93.98 82.55 0)
 			(effects
@@
 			(project "power"
 				(path "/b905a668-e7ff-483f-a1a5-78bb0590864b/f3b54294-78cd-476f-bb66-930d59da1e95"
-					(reference "#PWR040")
+					(reference "#PWR042")
 					(unit 1)
 				)
@@
 		(dnp no)
 		(fields_autoplaced yes)
-		(property "Reference" "#PWR042"
+		(property "Reference" "#PWR044"
 			(at 97.79 146.05 0)
 			(effects
@@
 			(project "power"
 				(path "/b905a668-e7ff-483f-a1a5-78bb0590864b/f3b54294-78cd-476f-bb66-930d59da1e95"
-					(reference "#PWR042")
+					(reference "#PWR044")
 					(unit 1)
 				)
@@
 		(on_board yes)
 		(dnp no)
-		(property "Reference" "#PWR058"
+		(property "Reference" "#PWR060"
 			(at 176.53 69.85 0)
 			(effects
@@
 			(project "power"
 				(path "/b905a668-e7ff-483f-a1a5-78bb0590864b/f3b54294-78cd-476f-bb66-930d59da1e95"
-					(reference "#PWR058")
+					(reference "#PWR060")
 					(unit 1)
 				)
@@
 		(dnp no)
 		(fields_autoplaced yes)
-		(property "Reference" "J14"
+		(property "Reference" "J13"
 			(at 248.92 106.6799 0)
 			(effects
@@
 			(project "power"
 				(path "/b905a668-e7ff-483f-a1a5-78bb0590864b/f3b54294-78cd-476f-bb66-930d59da1e95"
-					(reference "J14")
+					(reference "J13")
 					(unit 1)
 				)
@@
 		(dnp no)
 		(fields_autoplaced yes)
-		(property "Reference" "#PWR038"
+		(property "Reference" "#PWR040"
 			(at 85.09 146.05 0)
 			(effects
@@
 			(project "power"
 				(path "/b905a668-e7ff-483f-a1a5-78bb0590864b/f3b54294-78cd-476f-bb66-930d59da1e95"
-					(reference "#PWR038")
+					(reference "#PWR040")
 					(unit 1)
 				)
@@
 		(dnp no)
 		(fields_autoplaced yes)
-		(property "Reference" "#PWR049"
+		(property "Reference" "#PWR051"
 			(at 128.27 144.78 0)
 			(effects
@@
 			(project "power"
 				(path "/b905a668-e7ff-483f-a1a5-78bb0590864b/f3b54294-78cd-476f-bb66-930d59da1e95"
-					(reference "#PWR049")
-					(unit 1)
-				)
+					(reference "#PWR051")
+					(unit 1)
+				)
