File: power/ELE_ANP.kicad_sch (KiCad schematic)
At the start: 11 parts, among them U8 LT6106

Commit message: 2026/04/01
Parts:
- D6: footprint SamacSys_Parts:SOD2512X110N -> footprints:SOD2512X110N
- R16, R17: footprint LED_SMD:LED_0805_2012Metric -> Resistor_SMD:R_0805_2012Metric
Changed lines of the file:
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@@
 		(dnp no)
 		(fields_autoplaced yes)
-		(property "Reference" "#PWR084"
+		(property "Reference" "#PWR086"
 			(at 128.27 125.73 0)
 			(effects
@@
 			(project "power"
 				(path "/b905a668-e7ff-483f-a1a5-78bb0590864b/b2880fc9-ffe6-470a-8ca0-b35b55d83219"
-					(reference "#PWR084")
+					(reference "#PWR086")
 					(unit 1)
 				)
@@
 		(dnp no)
 		(fields_autoplaced yes)
-		(property "Reference" "#PWR083"
+		(property "Reference" "#PWR085"
 			(at 116.84 93.98 0)
 			(effects
@@
 			(project "power"
 				(path "/b905a668-e7ff-483f-a1a5-78bb0590864b/b2880fc9-ffe6-470a-8ca0-b35b55d83219"
-					(reference "#PWR083")
+					(reference "#PWR085")
 					(unit 1)
 				)
@@
 		(dnp no)
 		(fields_autoplaced yes)
-		(property "Reference" "#PWR082"
+		(property "Reference" "#PWR084"
 			(at 71.12 125.73 0)
 			(effects
@@
 			(project "power"
 				(path "/b905a668-e7ff-483f-a1a5-78bb0590864b/b2880fc9-ffe6-470a-8ca0-b35b55d83219"
-					(reference "#PWR082")
+					(reference "#PWR084")
 					(unit 1)
 				)
@@
 			)
 		)
-		(property "Footprint" "LED_SMD:LED_0805_2012Metric"
+		(property "Footprint" "Resistor_SMD:R_0805_2012Metric"
 			(at 77.47 80.772 90)
 			(effects
@@
 		(dnp no)
 		(fields_autoplaced yes)
-		(property "Reference" "#PWR081"
+		(property "Reference" "#PWR083"
 			(at 57.15 57.15 0)
 			(effects
@@
 			(project "power"
 				(path "/b905a668-e7ff-483f-a1a5-78bb0590864b/b2880fc9-ffe6-470a-8ca0-b35b55d83219"
-					(reference "#PWR081")
+					(reference "#PWR083")
 					(unit 1)
 				)
@@
 		(on_board yes)
 		(dnp no)
-		(fields_autoplaced yes)
 		(property "Reference" "D4"
-			(at 121.92 111.76 0)
+			(at 124.968 111.76 0)
 			(effects
 				(font
@@
 		)
 		(property "Value" "D_Zener 3V"
-			(at 124.46 111.76 0)
+			(at 124.714 119.38 0)
 			(effects
 				(font
@@
 			)
 		)
-		(property "Footprint" "SamacSys_Parts:SOD2512X110N"
+		(property "Footprint" "footprints:SOD2512X110N"
 			(at 54.94 120.65 0)
 			(effects
@@
 		(dnp no)
 		(fields_autoplaced yes)
-		(property "Reference" "#PWR085"
+		(property "Reference" "#PWR087"
 			(at 148.59 134.62 0)
 			(effects
@@
 			(project "power"
 				(path "/b905a668-e7ff-483f-a1a5-78bb0590864b/b2880fc9-ffe6-470a-8ca0-b35b55d83219"
-					(reference "#PWR085")
+					(reference "#PWR087")
 					(unit 1)
 				)
@@
 			)
 		)
-		(property "Footprint" "LED_SMD:LED_0805_2012Metric"
+		(property "Footprint" "Resistor_SMD:R_0805_2012Metric"
 			(at 77.47 68.072 90)
 			(effects
