File: power/LAD_ANP.kicad_sch (KiCad schematic)
At the start: 11 parts, among them U9 LT6106

Commit message: 2026/04/01
Parts:
- D9: footprint SamacSys_Parts:SOD2512X110N -> footprints:SOD2512X110N
Changed lines of the file:
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@@
 		(dnp no)
 		(fields_autoplaced yes)
-		(property "Reference" "#PWR086"
+		(property "Reference" "#PWR088"
 			(at 72.39 52.07 0)
 			(effects
@@
 			(project "power"
 				(path "/b905a668-e7ff-483f-a1a5-78bb0590864b/4831bb9e-fd38-4fae-8ef4-b85584d1912a"
-					(reference "#PWR086")
+					(reference "#PWR088")
 					(unit 1)
 				)
@@
 		(dnp no)
 		(fields_autoplaced yes)
-		(property "Reference" "#PWR088"
+		(property "Reference" "#PWR090"
 			(at 132.08 88.9 0)
 			(effects
@@
 			(project "power"
 				(path "/b905a668-e7ff-483f-a1a5-78bb0590864b/4831bb9e-fd38-4fae-8ef4-b85584d1912a"
-					(reference "#PWR088")
+					(reference "#PWR090")
 					(unit 1)
 				)
@@
 		(dnp no)
 		(fields_autoplaced yes)
-		(property "Reference" "#PWR089"
+		(property "Reference" "#PWR091"
 			(at 143.51 120.65 0)
 			(effects
@@
 			(project "power"
 				(path "/b905a668-e7ff-483f-a1a5-78bb0590864b/4831bb9e-fd38-4fae-8ef4-b85584d1912a"
-					(reference "#PWR089")
+					(reference "#PWR091")
 					(unit 1)
 				)
@@
 		(dnp no)
 		(fields_autoplaced yes)
-		(property "Reference" "#PWR087"
+		(property "Reference" "#PWR089"
 			(at 86.36 120.65 0)
 			(effects
@@
 			(project "power"
 				(path "/b905a668-e7ff-483f-a1a5-78bb0590864b/4831bb9e-fd38-4fae-8ef4-b85584d1912a"
-					(reference "#PWR087")
+					(reference "#PWR089")
 					(unit 1)
 				)
@@
 		(dnp no)
 		(fields_autoplaced yes)
-		(property "Reference" "#PWR090"
+		(property "Reference" "#PWR092"
 			(at 163.83 129.54 0)
 			(effects
@@
 			(project "power"
 				(path "/b905a668-e7ff-483f-a1a5-78bb0590864b/4831bb9e-fd38-4fae-8ef4-b85584d1912a"
-					(reference "#PWR090")
+					(reference "#PWR092")
 					(unit 1)
 				)
@@
 			)
 		)
-		(property "Footprint" "SamacSys_Parts:SOD2512X110N"
+		(property "Footprint" "footprints:SOD2512X110N"
 			(at 70.18 115.57 0)
 			(effects
