File: power/power.kicad_sch (KiCad schematic)
At the start: 17 parts, among them J1 ELE, J10 Conn_01x06, J11 L_HAT_GEAR, J12 PWM_SPARE2, J2 LAD, J4 PIROT, J5 RJ45_logger, J6 RJ45_base, J7 RJ45_tail, J8 R_HAT_GEAR, J9 PWM_SPARE1

Commit message: 2026/04/01
Parts:
- J5: renamed from J10; footprint (none) -> Connector_JST:JST_XH_B6B-XH-AM_1x06_P2.50mm_Vertical
- renumbered J12 to J10, J7 to J11, J5 to J3, J8 to J6, J9 to J7, J6 to J8, J11 to J9
