File: power/_autosave-power.kicad_sch (KiCad schematic)
At the start: 17 parts, among them J1 ELE, J10 PWM_SPARE2, J11 RJ45_tail, J2 LAD, J3 RJ45_logger, J4 PIROT, J5 Conn_01x06, J6 R_HAT_GEAR, J7 PWM_SPARE1, J8 RJ45_base, J9 L_HAT_GEAR

Commit message: 2026/04/05
Parts:
- removed R1, R2: 100, Resistor_SMD:R_0805_2012Metric, symbol Device:R
Connections:
- net ELE: now also J1.1 (Pin_1)
- net LAD: now also J2.1 (Pin_1)
Changed lines of the file:
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@@
 	(wire
 		(pts
-			(xy 27.94 90.17) (xy 30.48 90.17)
+			(xy 27.94 90.17) (xy 45.72 90.17)
 		)
 		(stroke
@@
 	(wire
 		(pts
-			(xy 45.72 90.17) (xy 38.1 90.17)
-		)
-		(stroke
-			(width 0)
-			(type default)
-		)
-	)
-	(wire
-		(pts
-			(xy 27.94 59.69) (xy 31.75 59.69)
+			(xy 27.94 59.69) (xy 48.26 59.69)
 		)
 		(stroke
@@
 	(wire
 		(pts
-			(xy 48.26 59.69) (xy 39.37 59.69)
-		)
-		(stroke
-			(width 0)
-			(type default)
-		)
-	)
-	(wire
-		(pts
 			(xy 80.01 87.63) (xy 92.71 87.63)
 		)
@@
 	)
 	(symbol
-		(lib_id "Device:R")
-		(at 34.29 90.17 90)
-		(unit 1)
-		(exclude_from_sim no)
-		(in_bom yes)
-		(on_board yes)
-		(dnp no)
-		(fields_autoplaced yes)
-		(property "Reference" "R1"
-			(at 34.29 83.82 90)
-			(effects
-				(font
-					(size 1.27 1.27)
-				)
-			)
-		)
-		(property "Value" "100"
-			(at 34.29 86.36 90)
-			(effects
-				(font
-					(size 1.27 1.27)
-				)
-			)
-		)
-		(property "Footprint" "Resistor_SMD:R_0805_2012Metric"
-			(at 34.29 91.948 90)
-			(effects
-				(font
-					(size 1.27 1.27)
-				)
-				(hide yes)
-			)
-		)
-		(property "Datasheet" "~"
-			(at 34.29 90.17 0)
-			(effects
-				(font
-					(size 1.27 1.27)
-				)
-				(hide yes)
-			)
-		)
-		(property "Description" "Resistor"
-			(at 34.29 90.17 0)
-			(effects
-				(font
-					(size 1.27 1.27)
-				)
-				(hide yes)
-			)
-		)
-		(pin "1"
-		)
-		(pin "2"
-		)
-		(instances
-			(project "power"
-				(path "/b905a668-e7ff-483f-a1a5-78bb0590864b"
-					(reference "R1")
-					(unit 1)
-				)
-			)
-		)
-	)
-	(symbol
 		(lib_id "power:GND")
 		(at 222.25 132.08 90)
@@
 					(unit 1)
 				)
-			)
-		)
-	)
-	(symbol
-		(lib_id "Device:R")
-		(at 35.56 59.69 270)
-		(unit 1)
-		(exclude_from_sim no)
-		(in_bom yes)
-		(on_board yes)
-		(dnp no)
-		(fields_autoplaced yes)
-		(property "Reference" "R2"
-			(at 35.56 53.34 90)
-			(effects
-				(font
-					(size 1.27 1.27)
-				)
-			)
-		)
-		(property "Value" "100"
-			(at 35.56 55.88 90)
-			(effects
-				(font
-					(size 1.27 1.27)
-				)
-			)
-		)
-		(property "Footprint" "Resistor_SMD:R_0805_2012Metric"
-			(at 35.56 57.912 90)
-			(effects
-				(font
-					(size 1.27 1.27)
-				)
-				(hide yes)
-			)
-		)
-		(property "Datasheet" "~"
-			(at 35.56 59.69 0)
-			(effects
-				(font
-					(size 1.27 1.27)
-				)
-				(hide yes)
-			)
-		)
-		(property "Description" "Resistor"
-			(at 35.56 59.69 0)
-			(effects
-				(font
-					(size 1.27 1.27)
-				)
-				(hide yes)
-			)
-		)
-		(pin "2"
-		)
-		(pin "1"
-		)
-		(instances
-			(project "power"
-				(path "/b905a668-e7ff-483f-a1a5-78bb0590864b"
-					(reference "R2")
-					(unit 1)
-				)
