File: power/power_.kicad_sch (KiCad schematic)
At the start: 14 parts, among them J15 電源入力, U4 NCP1117-5.0_SOT223, U5 NCP1117-5.0_SOT223, U6 NCP1117-5.0_SOT223, U7 NCP1117-5.0_SOT223

Commit message: 2026/04/01
Parts:
- D3: footprint (none) -> Diode_SMD:D_SMA
- renumbered J15 to J14
Changed lines of the file:
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@@
 		(dnp no)
 		(fields_autoplaced yes)
-		(property "Reference" "#PWR069"
+		(property "Reference" "#PWR071"
 			(at 73.66 97.79 0)
 			(effects
@@
 			(project "power"
 				(path "/b905a668-e7ff-483f-a1a5-78bb0590864b/80697437-fc60-4acb-ac74-8e2ba3308822"
-					(reference "#PWR069")
+					(reference "#PWR071")
 					(unit 1)
 				)
@@
 		(dnp no)
 		(fields_autoplaced yes)
-		(property "Reference" "#PWR074"
+		(property "Reference" "#PWR076"
 			(at 92.71 123.19 0)
 			(effects
@@
 			(project "power"
 				(path "/b905a668-e7ff-483f-a1a5-78bb0590864b/80697437-fc60-4acb-ac74-8e2ba3308822"
-					(reference "#PWR074")
+					(reference "#PWR076")
 					(unit 1)
 				)
@@
 		(on_board yes)
 		(dnp no)
-		(property "Reference" "#PWR073"
+		(property "Reference" "#PWR075"
 			(at 92.71 97.79 0)
 			(effects
@@
 			(project "power"
 				(path "/b905a668-e7ff-483f-a1a5-78bb0590864b/80697437-fc60-4acb-ac74-8e2ba3308822"
-					(reference "#PWR073")
+					(reference "#PWR075")
 					(unit 1)
 				)
@@
 		(dnp no)
 		(fields_autoplaced yes)
-		(property "Reference" "#PWR075"
+		(property "Reference" "#PWR077"
 			(at 92.71 149.86 0)
 			(effects
@@
 			(project "power"
 				(path "/b905a668-e7ff-483f-a1a5-78bb0590864b/80697437-fc60-4acb-ac74-8e2ba3308822"
-					(reference "#PWR075")
+					(reference "#PWR077")
 					(unit 1)
 				)
@@
 		(dnp no)
 		(fields_autoplaced yes)
-		(property "Reference" "#PWR072"
+		(property "Reference" "#PWR074"
 			(at 74.93 73.66 0)
 			(effects
@@
 			(project "power"
 				(path "/b905a668-e7ff-483f-a1a5-78bb0590864b/80697437-fc60-4acb-ac74-8e2ba3308822"
-					(reference "#PWR072")
+					(reference "#PWR074")
 					(unit 1)
 				)
@@
 		(dnp no)
 		(fields_autoplaced yes)
-		(property "Reference" "#PWR070"
+		(property "Reference" "#PWR072"
 			(at 73.66 123.19 0)
 			(effects
@@
 			(project "power"
 				(path "/b905a668-e7ff-483f-a1a5-78bb0590864b/80697437-fc60-4acb-ac74-8e2ba3308822"
-					(reference "#PWR070")
+					(reference "#PWR072")
 					(unit 1)
 				)
@@
 		(dnp no)
 		(fields_autoplaced yes)
-		(property "Reference" "#PWR067"
+		(property "Reference" "#PWR069"
 			(at 45.72 68.58 0)
 			(effects
@@
 			(project "power"
 				(path "/b905a668-e7ff-483f-a1a5-78bb0590864b/80697437-fc60-4acb-ac74-8e2ba3308822"
-					(reference "#PWR067")
+					(reference "#PWR069")
 					(unit 1)
 				)
@@
 		(dnp no)
 		(fields_autoplaced yes)
-		(property "Reference" "#PWR079"
+		(property "Reference" "#PWR081"
 			(at 104.14 149.86 0)
 			(effects
@@
 			(project "power"
 				(path "/b905a668-e7ff-483f-a1a5-78bb0590864b/80697437-fc60-4acb-ac74-8e2ba3308822"
-					(reference "#PWR079")
+					(reference "#PWR081")
 					(unit 1)
 				)
@@
 		(dnp no)
 		(fields_autoplaced yes)
-		(property "Reference" "#PWR076"
+		(property "Reference" "#PWR078"
 			(at 93.98 73.66 0)
 			(effects
@@
 			(project "power"
 				(path "/b905a668-e7ff-483f-a1a5-78bb0590864b/80697437-fc60-4acb-ac74-8e2ba3308822"
-					(reference "#PWR076")
+					(reference "#PWR078")
 					(unit 1)
 				)
@@
 		(dnp no)
 		(fields_autoplaced yes)
-		(property "Reference" "J15"
+		(property "Reference" "J14"
 			(at 35.56 69.85 0)
 			(effects
@@
 			(project "power"
 				(path "/b905a668-e7ff-483f-a1a5-78bb0590864b/80697437-fc60-4acb-ac74-8e2ba3308822"
-					(reference "J15")
+					(reference "J14")
 					(unit 1)
 				)
@@
 		(dnp no)
 		(fields_autoplaced yes)
-		(property "Reference" "#PWR071"
+		(property "Reference" "#PWR073"
 			(at 73.66 149.86 0)
 			(effects
@@
 			(project "power"
 				(path "/b905a668-e7ff-483f-a1a5-78bb0590864b/80697437-fc60-4acb-ac74-8e2ba3308822"
-					(reference "#PWR071")
+					(reference "#PWR073")
 					(unit 1)
 				)
@@
 		(dnp no)
 		(fields_autoplaced yes)
-		(property "Reference" "#PWR068"
+		(property "Reference" "#PWR070"
 			(at 48.26 85.09 0)
 			(effects
@@
 			(project "power"
 				(path "/b905a668-e7ff-483f-a1a5-78bb0590864b/80697437-fc60-4acb-ac74-8e2ba3308822"
-					(reference "#PWR068")
+					(reference "#PWR070")
 					(unit 1)
 				)
@@
 		(dnp no)
 		(fields_autoplaced yes)
-		(property "Reference" "#PWR077"
+		(property "Reference" "#PWR079"
 			(at 104.14 97.79 0)
 			(effects
@@
 			(project "power"
 				(path "/b905a668-e7ff-483f-a1a5-78bb0590864b/80697437-fc60-4acb-ac74-8e2ba3308822"
-					(reference "#PWR077")
+					(reference "#PWR079")
 					(unit 1)
 				)
@@
 			)
 		)
-		(property "Footprint" ""
+		(property "Footprint" "Diode_SMD:D_SMA"
 			(at 45.72 71.12 0)
 			(effects
@@
 		(dnp no)
 		(fields_autoplaced yes)
-		(property "Reference" "#PWR080"
+		(property "Reference" "#PWR082"
 			(at 105.41 73.66 0)
 			(effects
@@
 			(project "power"
 				(path "/b905a668-e7ff-483f-a1a5-78bb0590864b/80697437-fc60-4acb-ac74-8e2ba3308822"
-					(reference "#PWR080")
+					(reference "#PWR082")
 					(unit 1)
 				)
@@
 		(dnp no)
 		(fields_autoplaced yes)
-		(property "Reference" "#PWR078"
+		(property "Reference" "#PWR080"
 			(at 104.14 123.19 0)
 			(effects
@@
 			(project "power"
 				(path "/b905a668-e7ff-483f-a1a5-78bb0590864b/80697437-fc60-4acb-ac74-8e2ba3308822"
-					(reference "#PWR078")
-					(unit 1)
-				)
+					(reference "#PWR080")
+					(unit 1)
+				)

Commit message: 2026/04/05
Parts:
- D3: footprint Diode_SMD:D_SMA -> Diode_THT:D_P600_R-6_P7.62mm_Vertical_AnodeUp
Connections:
- net +8V: now also C30.1, C31.1, C32.1, C33.1, U4.3 (VI), U5.3 (VI), U6.3 (VI), U7.3 (VI)
- new net: D3.2 (A), J14.2 (Pin_2)
Other:
- moved on the sheet: D3
Changed lines of the file:
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@@
-	)
-	(junction
-		(at 54.61 76.2)
-		(diameter 0)
-		(color 0 0 0 0)
 	)
 	(junction
@@
 	)
 	(junction
-		(at 45.72 76.2)
+		(at 59.69 76.2)
 		(diameter 0)
 		(color 0 0 0 0)
@@
 	(wire
 		(pts
-			(xy 54.61 76.2) (xy 66.04 76.2)
-		)
-		(stroke
-			(width 0)
-			(type default)
-		)
-	)
-	(wire
-		(pts
 			(xy 66.04 59.69) (xy 74.93 59.69)
 		)
@@
 	(wire
 		(pts
+			(xy 59.69 76.2) (xy 66.04 76.2)
+		)
+		(stroke
+			(width 0)
+			(type default)
+		)
+	)
+	(wire
+		(pts
 			(xy 66.04 76.2) (xy 66.04 83.82)
 		)
@@
 	(wire
 		(pts
-			(xy 40.64 76.2) (xy 45.72 76.2)
+			(xy 40.64 76.2) (xy 41.91 76.2)
 		)
 		(stroke
@@
 	(wire
 		(pts
-			(xy 45.72 64.77) (xy 45.72 67.31)
-		)
-		(stroke
-			(width 0)
-			(type default)
-		)
-	)
-	(wire
-		(pts
 			(xy 66.04 135.89) (xy 73.66 135.89)
 		)
@@
 	(wire
 		(pts
-			(xy 45.72 76.2) (xy 54.61 76.2)
-		)
-		(stroke
-			(width 0)
-			(type default)
-		)
-	)
-	(wire
-		(pts
-			(xy 45.72 74.93) (xy 45.72 76.2)
-		)
-		(stroke
-			(width 0)
-			(type default)
-		)
-	)
-	(wire
-		(pts
 			(xy 66.04 76.2) (xy 66.04 59.69)
 		)
@@
 		(pts
 			(xy 104.14 77.47) (xy 104.14 83.82)
+		)
+		(stroke
+			(width 0)
+			(type default)
+		)
+	)
+	(wire
+		(pts
+			(xy 49.53 76.2) (xy 59.69 76.2)
 		)
 		(stroke
@@
 	)
 	(symbol
-		(lib_id "power:PWR_FLAG")
-		(at 54.61 76.2 0)
-		(unit 1)
-		(exclude_from_sim no)
-		(in_bom yes)
-		(on_board yes)
-		(dnp no)
-		(fields_autoplaced yes)
-		(property "Reference" "#FLG05"
-			(at 54.61 74.295 0)
-			(effects
-				(font
-					(size 1.27 1.27)
-				)
-				(hide yes)
-			)
-		)
-		(property "Value" "PWR_FLAG"
-			(at 54.61 71.12 0)
-			(effects
-				(font
-					(size 1.27 1.27)
-				)
-			)
-		)
-		(property "Footprint" ""
-			(at 54.61 76.2 0)
-			(effects
-				(font
-					(size 1.27 1.27)
-				)
-				(hide yes)
-			)
-		)
-		(property "Datasheet" "~"
-			(at 54.61 76.2 0)
-			(effects
-				(font
-					(size 1.27 1.27)
-				)
-				(hide yes)
-			)
-		)
-		(property "Description" "Special symbol for telling ERC where power comes from"
-			(at 54.61 76.2 0)
-			(effects
-				(font
-					(size 1.27 1.27)
-				)
-				(hide yes)
-			)
-		)
-		(pin "1"
-		)
-		(instances
-			(project "power"
-				(path "/b905a668-e7ff-483f-a1a5-78bb0590864b/80697437-fc60-4acb-ac74-8e2ba3308822"
-					(reference "#FLG05")
-					(unit 1)
-				)
-			)
-		)
-	)
-	(symbol
 		(lib_id "Regulator_Linear:NCP1117-5.0_SOT223")
 		(at 92.71 109.22 0)
@@
 	(symbol
 		(lib_id "power:+8V")
-		(at 45.72 64.77 0)
+		(at 59.69 76.2 0)
 		(unit 1)
 		(exclude_from_sim no)
@@
 		(fields_autoplaced yes)
 		(property "Reference" "#PWR069"
-			(at 45.72 68.58 0)
+			(at 59.69 80.01 0)
 			(effects
 				(font
@@
 		)
 		(property "Value" "+8V"
-			(at 45.72 59.69 0)
+			(at 59.69 71.12 0)
 			(effects
 				(font
@@
 		)
 		(property "Footprint" ""
-			(at 45.72 64.77 0)
+			(at 59.69 76.2 0)
 			(effects
 				(font
@@
 		)
 		(property "Datasheet" ""
-			(at 45.72 64.77 0)
+			(at 59.69 76.2 0)
 			(effects
 				(font
@@
 		)
 		(property "Description" "Power symbol creates a global label with name \"+8V\""
-			(at 45.72 64.77 0)
+			(at 59.69 76.2 0)
 			(effects
 				(font
@@
 	(symbol
 		(lib_id "Device:D")
-		(at 45.72 71.12 270)
+		(at 45.72 76.2 180)
 		(unit 1)
 		(exclude_from_sim no)
@@
 		(fields_autoplaced yes)
 		(property "Reference" "D3"
-			(at 48.26 69.8499 90)
-			(effects
-				(font
-					(size 1.27 1.27)
-				)
-				(justify left)
+			(at 45.72 69.85 0)
+			(effects
+				(font
+					(size 1.27 1.27)
+				)
 			)
 		)
 		(property "Value" "D"
-			(at 48.26 72.3899 90)
-			(effects
-				(font
-					(size 1.27 1.27)
-				)
-				(justify left)
-			)
-		)
-		(property "Footprint" "Diode_SMD:D_SMA"
-			(at 45.72 71.12 0)
+			(at 45.72 72.39 0)
+			(effects
+				(font
+					(size 1.27 1.27)
+				)
+			)
+		)
+		(property "Footprint" "Diode_THT:D_P600_R-6_P7.62mm_Vertical_AnodeUp"
+			(at 45.72 76.2 0)
 			(effects
 				(font
@@
 		)
 		(property "Datasheet" "~"
-			(at 45.72 71.12 0)
+			(at 45.72 76.2 0)
 			(effects
 				(font
@@
 		)
 		(property "Description" "Diode"
-			(at 45.72 71.12 0)
+			(at 45.72 76.2 0)
 			(effects
 				(font
@@
 		)
 		(property "Sim.Device" "D"
-			(at 45.72 71.12 0)
+			(at 45.72 76.2 0)
 			(effects
 				(font
@@
 		)
 		(property "Sim.Pins" "1=K 2=A"
-			(at 45.72 71.12 0)
-			(effects
-				(font
+			(at 45.72 76.2 0)
+			(effects
+				(font
