File: power/power.kicad_pcb (KiCad board)
At the start: 2 copper layers, 91.3 x 86.7 mm, 80 parts, among them IC1 W25Q128JVSIQTR, IC2 TJA1050T, J1 ELE, J10 PWM_SPARE2, J11 RJ45_tail, J12 USB_B_Micro, J13 Conn_01x02, J14 電源入力, J2 LAD, J3 RJ45_logger, J4 PIROT, J5 Conn_01x06, J6 R_HAT_GEAR, J7 PWM_SPARE1, J8 RJ45_base, J9 L_HAT_GEAR, SW1 SW_Push, SW2 SW_Push, U1 NCP1117-3.3_SOT223, U2 MCP2515-xSO, U3 RP2350_60QFN, U4 NCP1117-5.0_SOT223, U5 NCP1117-5.0_SOT223, U6 NCP1117-5.0_SOT223, U7 NCP1117-5.0_SOT223, Y1 ABM8-272-T3, Y2 ABLS-8.000MHZ-12-B-4-Y-T

Commit message: 20260406
Parts:
- added D4: LED, Inductor_SMD:L_0603_1608Metric, F.Cu at (186.7, 64.2)
- J12: footprint Connector_USB:USB_Micro-B_Amphenol_10103594-0001LF_Horizontal -> footprints:101181940001LF
- moved J11 9.03 mm to (210.0, 78.5), turned to -90 degrees
- moved J3 7.07 mm to (166.8, 108.6), turned to 180 degrees
- moved J8 6.22 mm to (189.1, 108.5), turned to 180 degrees
- moved J12 1.40 mm to (178.1, 39.4)
- moved Y1 0.13 mm to (178.9, 74.0)
Connections:
- U3 pad 33: unconnected-(U3-GPIO21-Pad33) -> Net-(D4-A)
Routing:
- net GND: track 338.8 -> 299.0 mm
- net /CAN_L: track 122.9 -> 93.5 mm
- net /5V_base: track 24.3 -> 32.9 mm, vias 0 -> 2
- net /CAN_H: track 99.3 -> 107.2 mm
- net /5V_logger: track 30.4 -> 24.5 mm, vias 1 -> 0
- net Net-(D4-A): track 0.00 -> 3.13 mm
- net +5V: track 105.2 -> 107.1 mm
- net /rp2350A/USB_D+: track 11.0 -> 11.8 mm
- net /rp2350A/USB_D-: track 11.1 -> 11.9 mm
- net Net-(D1-A): track 3.67 -> 4.49 mm
