File: power/power.kicad_pcb (KiCad board)
At the start: 2 copper layers, 91.3 x 86.7 mm, 81 parts, among them IC1 W25Q128JVSIQTR, IC2 TJA1050T, J1 ELE, J10 PWM_SPARE2, J11 RJ45_tail, J12 USB_B_Micro, J13 Conn_01x02, J14 電源入力, J2 LAD, J3 RJ45_logger, J4 PIROT, J5 Conn_01x06, J6 R_HAT_GEAR, J7 PWM_SPARE1, J8 RJ45_base, J9 L_HAT_GEAR, SW1 SW_Push, SW2 SW_Push, U1 NCP1117-3.3_SOT223, U2 MCP2515-xSO, U3 RP2350_60QFN, U4 NCP1117-5.0_SOT223, U5 NCP1117-5.0_SOT223, U6 NCP1117-5.0_SOT223, U7 NCP1117-5.0_SOT223, Y1 ABM8-272-T3, Y2 ABLS-8.000MHZ-12-B-4-Y-T

Commit message: 20261001
Parts:
- removed J12: USB_B_Micro, footprints:101181940001LF
- added J15: ZX62M-B-5P, footprints:ZX62MB5P, F.Cu at (178.1, 29.2)
- moved D1 3.41 mm to (181.1, 44.3)
Routing:
- net GND: track 299.0 -> 307.9 mm
- net /rp2350A/USB_D+: track 11.8 -> 19.8 mm
- net /rp2350A/USB_D-: track 11.9 -> 19.9 mm
- net Net-(D1-A): track 4.49 -> 10.1 mm
- net +5V: track 107.1 -> 108.0 mm, vias 4 -> 6
Other:
- board size 91.3 x 86.7 mm -> 91.3 x 97 mm
