File: power/rp2350A.kicad_sch (KiCad schematic)
At the start: 39 parts, among them IC1 W25Q128JVSIQTR, J13 USB_B_Micro, SW1 SW_Push, SW2 SW_Push, U1 NCP1117-3.3_SOT223, U3 RP2350_60QFN, Y1 ABM8-272-T3

Commit message: 2026/04/01
Parts:
- renumbered J13 to J12
Connections:
- no-connect marks 3 -> 10

Commit message: 2026/04/05
Connections:
- net ELE_LOAD: no longer names the net of U3.41 (GPIO27_ADC1)
- net LAD_LOAD: no longer names the net of U3.40 (GPIO26_ADC0)
- no-connect marks 10 -> 12
Changed lines of the file:
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@@
+	)
+	(no_connect
+		(at 271.78 227.33)
+	)
+	(no_connect
+		(at 271.78 229.87)
 	)
 	(no_connect
@@
 		)
 	)
-	(hierarchical_label "ELE_LOAD"
-		(shape input)
-		(at 271.78 229.87 0)
-		(effects
-			(font
-				(size 1.27 1.27)
-			)
-			(justify left)
-		)
-	)
 	(hierarchical_label "R_HAT"
 		(shape input)
@@
 		(effects
 			(font
-				(size 1.27 1.27)
-			)
-			(justify left)
-		)
-	)
-	(hierarchical_label "LAD_LOAD"
-		(shape input)
-		(at 271.78 227.33 0)
-		(effects
-			(font

Commit message: 20260406
Parts:
- added D4: LED, Inductor_SMD:L_0603_1608Metric, symbol Device:LED
- J12: footprint Connector_USB:USB_Micro-B_Amphenol_10103594-0001LF_Horizontal -> footprints:101181940001LF
Connections:
- net GND: now also D4.1 (K)
- net at U3.33 (GPIO21): now also D4.2 (A)
- no-connect marks 12 -> 11
Changed lines of the file:
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@@
 	)
 	(no_connect
-		(at 271.78 212.09)
-	)
-	(no_connect
 		(at 271.78 176.53)
 	)
@@
 	(wire
 		(pts
+			(xy 287.02 212.09) (xy 290.83 212.09)
+		)
+		(stroke
+			(width 0)
+			(type default)
+		)
+	)
+	(wire
+		(pts
 			(xy 184.15 154.94) (xy 184.15 138.43)
 		)
@@
 	(wire
 		(pts
+			(xy 271.78 212.09) (xy 279.4 212.09)
+		)
+		(stroke
+			(width 0)
+			(type default)
+		)
+	)
+	(wire
+		(pts
 			(xy 135.89 45.72) (xy 135.89 46.99)
 		)
@@
 			)
 		)
-		(property "Footprint" "Connector_USB:USB_Micro-B_Amphenol_10103594-0001LF_Horizontal"
+		(property "Footprint" "footprints:101181940001LF"
 			(at 68.58 52.07 0)
 			(effects
@@
 	)
 	(symbol
+		(lib_id "Device:LED")
+		(at 283.21 212.09 180)
+		(unit 1)
+		(exclude_from_sim no)
+		(in_bom yes)
+		(on_board yes)
+		(dnp no)
+		(fields_autoplaced yes)
+		(property "Reference" "D4"
+			(at 284.7975 204.47 0)
+			(effects
+				(font
+					(size 1.27 1.27)
+				)
+			)
+		)
+		(property "Value" "LED"
+			(at 284.7975 207.01 0)
+			(effects
+				(font
+					(size 1.27 1.27)
+				)
+			)
+		)
+		(property "Footprint" "Inductor_SMD:L_0603_1608Metric"
+			(at 283.21 212.09 0)
+			(effects
+				(font
+					(size 1.27 1.27)
+				)
+				(hide yes)
+			)
+		)
+		(property "Datasheet" "~"
+			(at 283.21 212.09 0)
+			(effects
+				(font
+					(size 1.27 1.27)
+				)
+				(hide yes)
+			)
+		)
+		(property "Description" "Light emitting diode"
+			(at 283.21 212.09 0)
+			(effects
+				(font
+					(size 1.27 1.27)
+				)
+				(hide yes)
+			)
+		)
+		(property "Sim.Pins" "1=K 2=A"
+			(at 283.21 212.09 0)
+			(effects
+				(font
+					(size 1.27 1.27)
+				)
+				(hide yes)
+			)
+		)
+		(pin "1"
+		)
+		(pin "2"
+		)
+		(instances
+			(project ""
+				(path "/b905a668-e7ff-483f-a1a5-78bb0590864b/804ea999-e638-418f-aadd-6db0b4e241f6"
+					(reference "D4")
+					(unit 1)
+				)
+			)
+		)
+	)
+	(symbol
 		(lib_id "power:+5V")
 		(at 104.14 34.29 0)
@@
 					(unit 1)
 				)
+			)
+		)
+	)
+	(symbol
+		(lib_id "power:GND")
+		(at 290.83 212.09 90)
+		(unit 1)
+		(exclude_from_sim no)
+		(in_bom yes)
+		(on_board yes)
+		(dnp no)
+		(fields_autoplaced yes)
+		(property "Reference" "#PWR02"
+			(at 297.18 212.09 0)
+			(effects
+				(font
+					(size 1.27 1.27)
+				)
+				(hide yes)
+			)
+		)
+		(property "Value" "GND"
+			(at 294.64 212.0899 90)
+			(effects
+				(font
+					(size 1.27 1.27)
+				)
+				(justify right)
+			)
+		)
+		(property "Footprint" ""
+			(at 290.83 212.09 0)
+			(effects
+				(font
+					(size 1.27 1.27)
+				)
+				(hide yes)
+			)
+		)
+		(property "Datasheet" ""
+			(at 290.83 212.09 0)
+			(effects
+				(font
+					(size 1.27 1.27)
+				)
+				(hide yes)
+			)
+		)
+		(property "Description" "Power symbol creates a global label with name \"GND\" , ground"
+			(at 290.83 212.09 0)
+			(effects
+				(font
+					(size 1.27 1.27)
+				)
+				(hide yes)
+			)
+		)
+		(pin "1"
+		)
+		(instances
+			(project ""
+				(path "/b905a668-e7ff-483f-a1a5-78bb0590864b/804ea999-e638-418f-aadd-6db0b4e241f6"
+					(reference "#PWR02")
+					(unit 1)
+				)
