File: power/rp2350A.kicad_sch (KiCad schematic)
At the start: 40 parts, among them IC1 W25Q128JVSIQTR, J12 USB_B_Micro, SW1 SW_Push, SW2 SW_Push, U1 NCP1117-3.3_SOT223, U3 RP2350_60QFN, Y1 ABM8-272-T3

Commit message: 20261001
Parts:
- removed J12: USB_B_Micro, footprints:101181940001LF, symbol Connector:USB_B_Micro
- added J15: ZX62M-B-5P, footprints:ZX62MB5P, symbol ZX62M-B-5P:ZX62M-B-5P
Connections:
- net GND: now also J15.5, J15.MP1, J15.MP2, J15.MP3, J15.MP4, J15.MP5, J15.MP6
- net USB_D+: now also J15.3
- net USB_D-: now also J15.2
- net at D1.2 (A): now also J15.1
